File: BeagleV/BeagleV.kicad_pcb (KiCad board)
At the start: 0 parts

Commit message: Initial commit to working branch, Cloned from the gitlab repository
Parts:
- added ANT1: RFECA3216060A1T, BeagleV:RFECA3216060A1T, F.Cu at (146.2, 99.6)
- added C1: 100nF/10V, Capacitor_SMD:C_0201_0603Metric, B.Cu at (100.3, 52.7)
- added C10: 10uF/6.3V, Capacitor_SMD:C_0402_1005Metric, F.Cu at (86.5, 73.9)
- added C100: 22uF/10V, Capacitor_SMD:C_0603_1608Metric, F.Cu at (122.0, 96.0)
- added C101: 1uF/10V, Capacitor_SMD:C_0402_1005Metric, F.Cu at (123.2, 95.4)
- added C102: 100nF/10V, Capacitor_SMD:C_0201_0603Metric, B.Cu at (119.5, 93.2)
- added C103: 100nF/10V, Capacitor_SMD:C_0201_0603Metric, B.Cu at (119.1, 85.4)
- added C104: 100nF/10V, Capacitor_SMD:C_0201_0603Metric, B.Cu at (121.6, 88.8)
- added C105: 100nF/10V, Capacitor_SMD:C_0201_0603Metric, B.Cu at (119.5, 87.1)
- added C106: 100nF/10V, Capacitor_SMD:C_0201_0603Metric, B.Cu at (127.3, 80.7)
- added C107: 100nF/10V, Capacitor_SMD:C_0201_0603Metric, B.Cu at (121.8, 82.8)
- added C108: 100nF/10V, Capacitor_SMD:C_0201_0603Metric, B.Cu at (122.0, 79.2)
- added C109: 100nF/10V, Capacitor_SMD:C_0201_0603Metric, B.Cu at (120.3, 79.2)
- added C11: 100nF/10V, Capacitor_SMD:C_0201_0603Metric, F.Cu at (93.1, 72.0)
- added C110: 100nF/10V, Capacitor_SMD:C_0201_0603Metric, B.Cu at (120.8, 93.4)
- added C111: 10uF/6.3V, Capacitor_SMD:C_0402_1005Metric, F.Cu at (124.2, 95.4)
- added C112: 100nF/10V, Capacitor_SMD:C_0201_0603Metric, B.Cu at (101.3, 87.7)
- added C113: 100nF/10V, Capacitor_SMD:C_0201_0603Metric, B.Cu at (100.2, 88.2)
- added C114: 100nF/10V, Capacitor_SMD:C_0201_0603Metric, B.Cu at (107.7, 87.3)
- added C115: 100nF/10V, Capacitor_SMD:C_0201_0603Metric, B.Cu at (107.7, 88.3)
- added C116: 1uF/10V, Capacitor_SMD:C_0402_1005Metric, B.Cu at (106.4, 86.0)
- added C117: 100nF/10V, Capacitor_SMD:C_0201_0603Metric, B.Cu at (103.9, 84.7)
- added C118: 100nF/10V, Capacitor_SMD:C_0201_0603Metric, B.Cu at (104.8, 85.9)
- added C119: 100nF/10V, Capacitor_SMD:C_0201_0603Metric, B.Cu at (104.9, 84.3)
- added C12: 100nF/10V, Capacitor_SMD:C_0201_0603Metric, F.Cu at (93.1, 73.7)
- added C120: 22uF/10V, Capacitor_SMD:C_0603_1608Metric, B.Cu at (93.5, 101.5)
- added C121: 10uF/10V, Capacitor_SMD:C_0402_1005Metric, B.Cu at (94.8, 101.0)
- added C122: 10uF/10V, Capacitor_SMD:C_0402_1005Metric, B.Cu at (95.8, 101.0)
- added C123: 1uF/10V, Capacitor_SMD:C_0402_1005Metric, B.Cu at (96.8, 101.0)
- added C124: 100nF/10V, Capacitor_SMD:C_0201_0603Metric, B.Cu at (101.2, 86.5)
- added C125: 100nF/10V, Capacitor_SMD:C_0201_0603Metric, B.Cu at (99.8, 86.5)
- added C126: 100nF/10V, Capacitor_SMD:C_0201_0603Metric, B.Cu at (99.5, 87.2)
- added C127: 100nF/10V, Capacitor_SMD:C_0201_0603Metric, B.Cu at (98.2, 93.7)
- added C128: 100nF/10V, Capacitor_SMD:C_0201_0603Metric, B.Cu at (100.8, 90.3)
- added C129: 100nF/10V, Capacitor_SMD:C_0201_0603Metric, B.Cu at (99.4, 88.8)
- added C13: 100nF/10V, Capacitor_SMD:C_0201_0603Metric, F.Cu at (92.3, 75.5)
- added C130: 100nF/10V, Capacitor_SMD:C_0201_0603Metric, B.Cu at (99.3, 90.3)
- added C131: 100nF/10V, Capacitor_SMD:C_0201_0603Metric, B.Cu at (99.2, 92.2)
- added C132: 100nF/10V, Capacitor_SMD:C_0201_0603Metric, B.Cu at (99.9, 92.2)
- added C133: 1nF/10V, Capacitor_SMD:C_0402_1005Metric, B.Cu at (99.4, 85.7)
- added C134: 22uF/10V, Capacitor_SMD:C_0603_1608Metric, B.Cu at (97.0, 98.4)
- added C135: 10uF/10V, Capacitor_SMD:C_0402_1005Metric, B.Cu at (99.3, 98.5)
- added C136: 1uF/10V, Capacitor_SMD:C_0402_1005Metric, B.Cu at (98.3, 98.5)
- added C137: 100nF/10V, Capacitor_SMD:C_0201_0603Metric, B.Cu at (108.4, 84.9)
- added C138: 100nF/10V, Capacitor_SMD:C_0201_0603Metric, B.Cu at (105.8, 84.0)
- added C139: 100nF/10V, Capacitor_SMD:C_0201_0603Metric, B.Cu at (104.1, 93.0)
- added C14: 100nF/10V, Capacitor_SMD:C_0201_0603Metric, F.Cu at (89.8, 75.5)
- added C140: 100nF/10V, Capacitor_SMD:C_0201_0603Metric, B.Cu at (104.0, 83.9)
- added C141: 1nF/10V, Capacitor_SMD:C_0402_1005Metric, B.Cu at (104.4, 94.0)
- added C142: 22uF/10V, Capacitor_SMD:C_0603_1608Metric, B.Cu at (114.2, 100.0)
- added C143: 10uF/10V, Capacitor_SMD:C_0402_1005Metric, B.Cu at (111.9, 100.0)
- added C144: 0uF/10V, Capacitor_SMD:C_0402_1005Metric, B.Cu at (112.9, 100.0)
- added C145: 1uF/10V, Capacitor_SMD:C_0402_1005Metric, B.Cu at (110.9, 100.0)
- added C146: 100nF/10V, Capacitor_SMD:C_0201_0603Metric, B.Cu at (109.7, 85.5)
- added C147: 100nF/10V, Capacitor_SMD:C_0201_0603Metric, B.Cu at (110.0, 84.6)
- added C148: 100nF/10V, Capacitor_SMD:C_0201_0603Metric, B.Cu at (110.0, 86.7)
- added C149: 100nF/10V, Capacitor_SMD:C_0201_0603Metric, B.Cu at (110.7, 87.9)
- added C15: 100nF/10V, Capacitor_SMD:C_0201_0603Metric, F.Cu at (86.6, 75.0)
- added C150: 100nF/10V, Capacitor_SMD:C_0201_0603Metric, B.Cu at (109.0, 93.1)
- added C151: 100nF/10V, Capacitor_SMD:C_0201_0603Metric, B.Cu at (109.2, 92.3)
- added C152: 100nF/10V, Capacitor_SMD:C_0201_0603Metric, B.Cu at (109.6, 90.8)
- added C153: 100nF/10V, Capacitor_SMD:C_0201_0603Metric, B.Cu at (109.0, 88.2)
- added C154: 100nF/10V, Capacitor_SMD:C_0201_0603Metric, B.Cu at (108.4, 88.2)
- added C155: 1nF/10V, Capacitor_SMD:C_0402_1005Metric, B.Cu at (109.2, 93.9)
- added C156: 22uF/10V, Capacitor_SMD:C_0603_1608Metric, B.Cu at (100.8, 78.9)
- added C157: 22uF/10V, Capacitor_SMD:C_0603_1608Metric, B.Cu at (100.8, 80.7)
- added C158: 10uF/10V, Capacitor_SMD:C_0402_1005Metric, B.Cu at (98.1, 81.9)
- added C159: 10uF/10V, Capacitor_SMD:C_0402_1005Metric, B.Cu at (98.1, 78.9)
- added C16: 100nF/10V, Capacitor_SMD:C_0201_0603Metric, F.Cu at (86.5, 72.8)
- added C160: 1uF/10V, Capacitor_SMD:C_0402_1005Metric, B.Cu at (101.1, 84.9)
- added C161: 100nF/10V, Capacitor_SMD:C_0201_0603Metric, B.Cu at (107.4, 89.3)
- added C162: 100nF/10V, Capacitor_SMD:C_0201_0603Metric, B.Cu at (106.7, 87.5)
- added C163: 100nF/10V, Capacitor_SMD:C_0201_0603Metric, B.Cu at (102.3, 84.9)
- added C164: 100nF/10V, Capacitor_SMD:C_0201_0603Metric, B.Cu at (103.7, 86.2)
- added C165: 100nF/10V, Capacitor_SMD:C_0201_0603Metric, B.Cu at (102.3, 87.0)
- added C166: 100nF/10V, Capacitor_SMD:C_0201_0603Metric, B.Cu at (102.2, 86.2)
- added C167: 100nF/10V, Capacitor_SMD:C_0201_0603Metric, B.Cu at (102.3, 87.8)
- added C168: 100nF/10V, Capacitor_SMD:C_0201_0603Metric, B.Cu at (102.8, 88.8)
- added C169: 100nF/10V, Capacitor_SMD:C_0201_0603Metric, B.Cu at (104.4, 89.1)
- added C17: 100nF/10V, Capacitor_SMD:C_0201_0603Metric, F.Cu at (89.8, 69.0)
- added C170: 100nF/10V, Capacitor_SMD:C_0201_0603Metric, B.Cu at (105.8, 90.1)
- added C171: 100nF/10V, Capacitor_SMD:C_0201_0603Metric, B.Cu at (105.2, 90.1)
- added C172: 100nF/10V, Capacitor_SMD:C_0201_0603Metric, B.Cu at (107.0, 90.3)
- added C173: 100nF/10V, Capacitor_SMD:C_0201_0603Metric, B.Cu at (108.4, 90.5)
- added C174: 100nF/10V, Capacitor_SMD:C_0201_0603Metric, B.Cu at (106.1, 91.8)
- added C175: 100nF/10V, Capacitor_SMD:C_0201_0603Metric, B.Cu at (106.1, 91.0)
- added C176: 1nF/10V, Capacitor_SMD:C_0402_1005Metric, B.Cu at (108.0, 91.8)
- added C177: 10uF/6.3V, Capacitor_SMD:C_0402_1005Metric, B.Cu at (116.8, 97.8)
- added C178: 1uF/10V, Capacitor_SMD:C_0402_1005Metric, B.Cu at (106.4, 85.0)
- added C179: 100nF/10V, Capacitor_SMD:C_0201_0603Metric, B.Cu at (105.7, 92.8)
- added C18: 100nF/10V, Capacitor_SMD:C_0201_0603Metric, B.Cu at (91.4, 63.9)
- added C180: 100nF/10V, Capacitor_SMD:C_0201_0603Metric, B.Cu at (106.9, 92.9)
- added C181: 100nF/10V, Capacitor_SMD:C_0201_0603Metric, B.Cu at (104.5, 90.1)
- added C182: 1uF/10V, Capacitor_SMD:C_0402_1005Metric, B.Cu at (107.0, 94.8)
- added C183: 100nF/10V, Capacitor_SMD:C_0201_0603Metric, B.Cu at (107.7, 85.0)
- added C184: 100nF/10V, Capacitor_SMD:C_0201_0603Metric, B.Cu at (101.8, 89.1)
- added C185: 100nF/10V, Capacitor_SMD:C_0201_0603Metric, B.Cu at (94.8, 75.9)
- added C186: 100nF/10V, Capacitor_SMD:C_0201_0603Metric, B.Cu at (92.5, 77.9)
- added C187: 10uF/6.4V, Capacitor_SMD:C_0402_1005Metric, B.Cu at (116.8, 99.8)
- added C188: 1uF/10V, Capacitor_SMD:C_0402_1005Metric, B.Cu at (116.8, 100.7)
- added C189: 100nF/10V, Capacitor_SMD:C_0201_0603Metric, B.Cu at (108.3, 86.3)
- added C19: 100nF/10V, Capacitor_SMD:C_0201_0603Metric, B.Cu at (65.0, 76.4)
- added C190: 100nF/10V, Capacitor_SMD:C_0201_0603Metric, B.Cu at (106.7, 94.0)
- added C191: 100nF/10V, Capacitor_SMD:C_0201_0603Metric, B.Cu at (103.9, 90.1)
- added C192: 1uF/10V, Capacitor_SMD:C_0402_1005Metric, B.Cu at (116.8, 98.8)
- added C193: 100nF/10V, Capacitor_SMD:C_0201_0603Metric, B.Cu at (102.2, 90.3)
- added C194: 100nF/10V, Capacitor_SMD:C_0201_0603Metric, B.Cu at (103.2, 90.1)
- added C195: 100nF/10V, Capacitor_SMD:C_0201_0603Metric, B.Cu at (107.8, 93.7)
- added C196: DNP, Capacitor_SMD:C_0201_0603Metric, B.Cu at (105.1, 82.3)
- added C197: 100nF, Capacitor_SMD:C_0402_1005Metric, B.Cu at (99.8, 70.7)
- added C198: 1uF/10V, Capacitor_SMD:C_0402_1005Metric, F.Cu at (138.0, 87.6)
- added C199: 100nF/10V, Capacitor_SMD:C_0201_0603Metric, F.Cu at (138.0, 86.6)
- added C2: 100nF/10V1, Capacitor_SMD:C_0201_0603Metric, B.Cu at (93.8, 52.8)
- added C20: 100nF/10V, Capacitor_SMD:C_0201_0603Metric, F.Cu at (67.3, 72.0)
- added C200: 2.2uF/6.3V, Capacitor_SMD:C_0402_1005Metric, B.Cu at (89.8, 107.3)
- added C201: 100nF/10V, Capacitor_SMD:C_0201_0603Metric, B.Cu at (89.7, 108.6)
- added C202: 1uF/10V, Capacitor_SMD:C_0402_1005Metric, B.Cu at (99.0, 101.0)
- added C203: 100nF/10V, Capacitor_SMD:C_0201_0603Metric, B.Cu at (102.0, 92.2)
- added C204: 1uF/10V, Capacitor_SMD:C_0402_1005Metric, B.Cu at (98.1, 81.0)
- added C205: 100nF/10V, Capacitor_SMD:C_0201_0603Metric, B.Cu at (104.2, 87.3)
- added C206: 1uF/10V, Capacitor_SMD:C_0402_1005Metric, B.Cu at (100.0, 101.0)
- added C207: 100nF/10V, Capacitor_SMD:C_0201_0603Metric, B.Cu at (104.1, 92.3)
- added C208: 1uF/10V, Capacitor_SMD:C_0402_1005Metric, B.Cu at (108.2, 82.8)
- added C209: 100nF/10V, Capacitor_SMD:C_0201_0603Metric, B.Cu at (108.1, 84.0)
- added C21: 100uF/6.3V, Capacitor_SMD:C_1206_3216Metric, B.Cu at (67.0, 74.0)
- added C210: 100nF/10V, Capacitor_SMD:C_0201_0603Metric, B.Cu at (104.1, 91.6)
- added C211: 100nF/10V, Capacitor_SMD:C_0201_0603Metric, B.Cu at (102.1, 93.2)
- added C212: 100nF/10V, Capacitor_SMD:C_0201_0603Metric, B.Cu at (102.2, 84.1)
- added C213: 1pF/50V, Capacitor_SMD:C_0201_0603Metric, F.Cu at (145.1, 104.3)
- added C215: 10pF, Capacitor_SMD:C_0402_1005Metric, B.Cu at (105.5, 72.6)
- added C216: 1uF/10V, Capacitor_SMD:C_0402_1005Metric, B.Cu at (98.0, 101.0)
- added C217: 100nF/10V, Capacitor_SMD:C_0201_0603Metric, B.Cu at (103.1, 92.1)
- added C218: 1uF/10V, Capacitor_SMD:C_0402_1005Metric, B.Cu at (100.6, 82.0)
- added C219: 100nF/10V, Capacitor_SMD:C_0201_0603Metric, B.Cu at (105.2, 87.5)
- added C22: 10uF/6.3V, Capacitor_SMD:C_0402_1005Metric, B.Cu at (92.9, 65.4)
- added C220: 1uF/10V, Capacitor_SMD:C_0402_1005Metric, B.Cu at (98.1, 80.0)
- added C221: 100nF/10V, Capacitor_SMD:C_0201_0603Metric, B.Cu at (110.0, 83.9)
- added C222: 4.7uF/10V, Capacitor_SMD:C_0402_1005Metric, F.Cu at (136.2, 64.5)
- added C223: 10pF, Capacitor_SMD:C_0402_1005Metric, F.Cu at (103.5, 75.8)
- added C224: 10pF, Capacitor_SMD:C_0402_1005Metric, F.Cu at (105.8, 75.8)
- added C226: DNP, Capacitor_SMD:C_0201_0603Metric, F.Cu at (144.0, 103.9)
- added C227: 10nF/50V, Capacitor_SMD:C_0402_1005Metric, F.Cu at (146.2, 96.4)
- added C228: 1nF/2kV, Capacitor_SMD:C_1206_3216Metric, B.Cu at (88.3, 50.8)
- added C229: 100nF/10V, Capacitor_SMD:C_0201_0603Metric, B.Cu at (137.6, 101.5)
- added C23: 10uF/6.3V, Capacitor_SMD:C_0402_1005Metric, F.Cu at (86.7, 76.0)
- added C230: 10uF/6.3V, Capacitor_SMD:C_0402_1005Metric, B.Cu at (136.7, 101.5)
- added C231: 10uF/6.3V, Capacitor_SMD:C_0402_1005Metric, B.Cu at (135.8, 101.5)
- added C232: 10uF/6.3V, Capacitor_SMD:C_0402_1005Metric, F.Cu at (135.0, 93.6)
- added C233: 100nF/10V, Capacitor_SMD:C_0402_1005Metric, B.Cu at (129.4, 97.3)
- added C234: 1uF/10V, Capacitor_SMD:C_0402_1005Metric, B.Cu at (130.3, 97.6)
- added C235: 22pF/50V, Capacitor_SMD:C_0402_1005Metric, F.Cu at (139.0, 93.9)
- added C236: 22pF/50V, Capacitor_SMD:C_0402_1005Metric, F.Cu at (136.8, 92.8)
- added C237: 100nF/10V, Capacitor_SMD:C_0201_0603Metric, B.Cu at (93.3, 77.9)
- added C238: 100nF/10V, Capacitor_SMD:C_0201_0603Metric, B.Cu at (89.2, 78.0)
- added C239: 100nF/10V, Capacitor_SMD:C_0201_0603Metric, B.Cu at (90.0, 78.0)
- added C24: 100nF/10V, Capacitor_SMD:C_0201_0603Metric, B.Cu at (94.0, 75.9)
- added C240: 100nF/10V, Capacitor_SMD:C_0201_0603Metric, B.Cu at (87.7, 78.0)
- added C241: 100nF/10V, Capacitor_SMD:C_0201_0603Metric, B.Cu at (88.5, 78.0)
- added C242: 100nF/10V, Capacitor_SMD:C_0201_0603Metric, B.Cu at (95.8, 73.4)
- added C243: 100nF/10V, Capacitor_SMD:C_0201_0603Metric, B.Cu at (95.8, 72.7)
- added C244: 100nF/10V, Capacitor_SMD:C_0201_0603Metric, B.Cu at (95.8, 74.8)
- added C245: 100nF/10V, Capacitor_SMD:C_0201_0603Metric, B.Cu at (95.8, 74.1)
- added C246: 22pF, Capacitor_SMD:C_0402_1005Metric, B.Cu at (96.3, 66.7)
- added C247: 22pF, Capacitor_SMD:C_0402_1005Metric, B.Cu at (95.8, 71.8)
- added C248: 22uF/10V, Capacitor_SMD:C_0603_1608Metric, F.Cu at (131.4, 56.4)
- added C249: 10uF/10V, Capacitor_SMD:C_0603_1608Metric, B.Cu at (133.0, 61.4)
- added C25: 100nF/10V, Capacitor_SMD:C_0201_0603Metric, B.Cu at (68.5, 93.2)
- added C250: 100nF/10V, Capacitor_SMD:C_0402_1005Metric, B.Cu at (123.9, 58.4)
- added C26: 100uF/10V, Capacitor_SMD:C_1206_3216Metric, B.Cu at (66.8, 93.9)
- added C266: 2.2uF/6.3V, Capacitor_SMD:C_0402_1005Metric, B.Cu at (89.9, 101.4)
- added C267: 100nF/10V, Capacitor_SMD:C_0201_0603Metric, B.Cu at (89.9, 102.4)
- added C268: 2.2uF/10V, Capacitor_SMD:C_0402_1005Metric, B.Cu at (82.8, 102.0)
- added C269: 100nF/10V, Capacitor_SMD:C_0201_0603Metric, B.Cu at (82.8, 103.3)
- added C27: 22uF/10V, Capacitor_SMD:C_0603_1608Metric, B.Cu at (131.5, 56.6)
- added C270: 100nF/10V, Capacitor_SMD:C_0201_0603Metric, B.Cu at (82.8, 108.0)
- added C271: 2.2uF/6.3V, Capacitor_SMD:C_0402_1005Metric, B.Cu at (82.9, 109.0)
- added C272: 100nF/10V, Capacitor_SMD:C_0201_0603Metric, B.Cu at (141.7, 91.7)
- added C273: 22uF/10V, Capacitor_SMD:C_0603_1608Metric, B.Cu at (138.2, 64.0)
- added C274: 22uF/10V, Capacitor_SMD:C_0603_1608Metric, F.Cu at (138.9, 63.4)
- added C275: 22uF/10V, Capacitor_SMD:C_0603_1608Metric, F.Cu at (127.3, 56.4)
- added C276: 22uF/10V, Capacitor_SMD:C_0603_1608Metric, B.Cu at (127.2, 56.5)
- added C277: 100nF/10V, Capacitor_SMD:C_0201_0603Metric, F.Cu at (138.3, 65.8)
- added C278: 10uF/6.3V, Capacitor_SMD:C_0402_1005Metric, F.Cu at (128.0, 81.8)
- added C279: 100nF/10V, Capacitor_SMD:C_0201_0603Metric, F.Cu at (129.0, 81.9)
- added C28: 10uF/6.3V, Capacitor_SMD:C_0402_1005Metric, B.Cu at (112.4, 68.6)
- added C280: 10uF/6.3V, Capacitor_SMD:C_0402_1005Metric, F.Cu at (142.2, 60.6)
- added C281: 100nF/10V, Capacitor_SMD:C_0201_0603Metric, F.Cu at (141.1, 60.8)
- added C282: 100nF/10V, Capacitor_SMD:C_0201_0603Metric, F.Cu at (137.1, 74.2)
- added C283: 22uF/10V, Capacitor_SMD:C_0603_1608Metric, B.Cu at (127.4, 60.9)
- added C284: 22uF/10V, Capacitor_SMD:C_0603_1608Metric, B.Cu at (127.4, 62.4)
- added C286: 100nF/10V, Capacitor_SMD:C_0201_0603Metric, F.Cu at (122.3, 70.5)
- added C287: 100nF/10V, Capacitor_SMD:C_0201_0603Metric, F.Cu at (122.3, 72.1)
- added C288: 10uF/10V, Capacitor_SMD:C_0402_1005Metric, F.Cu at (125.0, 72.0)
- added C289: 2.2uF/10V, Capacitor_SMD:C_0603_1608Metric, B.Cu at (132.8, 65.3)
- added C29: 100nF/10V, Capacitor_SMD:C_0201_0603Metric, B.Cu at (112.3, 67.8)
- added C290: 2.2uF/10V, Capacitor_SMD:C_0603_1608Metric, B.Cu at (127.4, 63.9)
- added C291: 10uF/10V, Capacitor_SMD:C_0603_1608Metric, B.Cu at (132.9, 63.8)
- added C293: 10uF/10V, Capacitor_SMD:C_0603_1608Metric, B.Cu at (130.1, 62.1)
- added C294: 22uF/10V, Capacitor_SMD:C_0603_1608Metric, F.Cu at (141.4, 71.8)
- added C295: 22uF/10V, Capacitor_SMD:C_0603_1608Metric, F.Cu at (141.4, 70.2)
- added C296: 2.2uF/10V, Capacitor_SMD:C_0402_1005Metric, F.Cu at (124.9, 58.4)
- added C297: 100nF/10V, Capacitor_SMD:C_0201_0603Metric, F.Cu at (137.1, 73.5)
- added C298: 10uF/10V, Capacitor_SMD:C_0402_1005Metric, F.Cu at (137.1, 75.0)
- added C3: 100n/10V, Capacitor_SMD:C_0201_0603Metric, F.Cu at (121.3, 101.8)
- added C30: 100uF/4V, Capacitor_SMD:C_0402_1005Metric, B.Cu at (103.3, 62.9)
- added C300: 100nF/10V, Capacitor_SMD:C_0201_0603Metric, F.Cu at (126.8, 58.0)
- added C301: 2.2uF, Capacitor_SMD:C_0603_1608Metric, F.Cu at (129.1, 71.3)
- added C302: 1nF/50V, Capacitor_SMD:C_0402_1005Metric, B.Cu at (144.3, 62.5)
- added C303: 10uF, Capacitor_SMD:C_0603_1608Metric, B.Cu at (135.7, 59.9)
- added C304: 10uF/10V, Capacitor_SMD:C_0603_1608Metric, B.Cu at (143.1, 58.8)
- added C305: 100nF, Capacitor_SMD:C_0201_0603Metric, F.Cu at (126.9, 70.6)
- added C306: 4.7uF/10V, Capacitor_SMD:C_0402_1005Metric, F.Cu at (130.5, 70.8)
- added C307: 4.7uF/10V, Capacitor_SMD:C_0402_1005Metric, F.Cu at (127.8, 70.8)
- added C308: 2.2uF/10V, Capacitor_SMD:C_0603_1608Metric, B.Cu at (130.3, 67.7)
- added C309: 1uF/10V, Capacitor_SMD:C_0402_1005Metric, F.Cu at (82.6, 112.8)
- added C31: 100uF/4V, Capacitor_SMD:C_0402_1005Metric, B.Cu at (115.4, 64.8)
- added C310: 1uF/10V, Capacitor_SMD:C_0402_1005Metric, F.Cu at (82.6, 114.1)
- added C311: 10nF/50V, Capacitor_SMD:C_0402_1005Metric, F.Cu at (79.5, 110.3)
- added C312: 10nF/50V, Capacitor_SMD:C_0402_1005Metric, F.Cu at (79.5, 105.0)
- added C313: 10nF/50V, Capacitor_SMD:C_0402_1005Metric, F.Cu at (77.2, 110.3)
- added C314: 10nF/50V, Capacitor_SMD:C_0402_1005Metric, F.Cu at (77.2, 105.0)
- added C32: 10uF/6.3V, Capacitor_SMD:C_0402_1005Metric, B.Cu at (112.3, 65.4)
- added C33: 100nF/10V, Capacitor_SMD:C_0201_0603Metric, B.Cu at (112.3, 64.3)
- added C34: 10uF/6.3V, Capacitor_SMD:C_0402_1005Metric, B.Cu at (106.8, 64.1)
- added C35: 100nF/10V, Capacitor_SMD:C_0201_0603Metric, B.Cu at (106.7, 64.9)
- added C36: 10uF/6.3V, Capacitor_SMD:C_0402_1005Metric, B.Cu at (109.7, 63.8)
- added C37: 100nF/10V, Capacitor_SMD:C_0201_0603Metric, B.Cu at (110.7, 63.6)
- added C38: 10uF/6.3V, Capacitor_SMD:C_0402_1005Metric, F.Cu at (115.2, 67.5)
- added C39: 100nF/10V, Capacitor_SMD:C_0201_0603Metric, F.Cu at (115.2, 65.5)
- added C4: 10uF/6.3V, Capacitor_SMD:C_0402_1005Metric, B.Cu at (91.6, 65.5)
- added C40: 10nF/50V, Capacitor_SMD:C_0402_1005Metric, F.Cu at (115.2, 66.5)
- added C42: DNP, Capacitor_SMD:C_0402_1005Metric, B.Cu at (99.3, 76.4)
- added C43: 22pF/50V, Capacitor_SMD:C_0402_1005Metric, F.Cu at (117.1, 60.7)
- added C44: DNP, Capacitor_SMD:C_0402_1005Metric, B.Cu at (100.5, 62.8)
- added C45: 22pF/50V, Capacitor_SMD:C_0402_1005Metric, F.Cu at (117.1, 65.3)
- added C46: 10pF, Capacitor_SMD:C_0402_1005Metric, B.Cu at (112.6, 74.4)
- added C47: 100nF/10V, Capacitor_SMD:C_0402_1005Metric, F.Cu at (81.8, 54.2)
- added C48: 22uF, Capacitor_SMD:C_0603_1608Metric, B.Cu at (83.2, 98.6)
- added C49: 1uF/10V, Capacitor_SMD:C_0402_1005Metric, B.Cu at (85.5, 98.8)
- added C5: 100nF/10V, Capacitor_SMD:C_0201_0603Metric, F.Cu at (87.9, 69.0)
- added C50: 100nF/10V, Capacitor_SMD:C_0201_0603Metric, B.Cu at (87.3, 84.7)
- added C51: 100nF/10V, Capacitor_SMD:C_0201_0603Metric, B.Cu at (88.8, 96.9)
- added C52: 100nF/10V, Capacitor_SMD:C_0201_0603Metric, B.Cu at (87.4, 92.1)
- added C53: 100nF/10V, Capacitor_SMD:C_0201_0603Metric, B.Cu at (85.2, 97.3)
- added C54: 100nF/10V, Capacitor_SMD:C_0201_0603Metric, F.Cu at (89.8, 81.5)
- added C55: 100nF/10V, Capacitor_SMD:C_0201_0603Metric, B.Cu at (87.5, 93.8)
- added C56: 100nF/10V, Capacitor_SMD:C_0201_0603Metric, B.Cu at (88.1, 86.4)
- added C57: 100nF/10V, Capacitor_SMD:C_0201_0603Metric, B.Cu at (90.0, 86.7)
- added C58: 100nF/10V, Capacitor_SMD:C_0201_0603Metric, B.Cu at (89.6, 90.4)
- added C59: 10uF/6.4V, Capacitor_SMD:C_0402_1005Metric, B.Cu at (84.5, 98.8)
- added C6: 100nF/10V, Capacitor_SMD:C_0201_0603Metric, F.Cu at (86.5, 69.5)
- added C60: 10uF/6.4V, Capacitor_SMD:C_0402_1005Metric, B.Cu at (82.5, 92.1)
- added C61: 100nF/10V, Capacitor_SMD:C_0201_0603Metric, B.Cu at (82.5, 94.0)
- added C62: 100nF/10V, Capacitor_SMD:C_0201_0603Metric, B.Cu at (82.5, 85.8)
- added C63: 100nF/10V, Capacitor_SMD:C_0201_0603Metric, B.Cu at (92.6, 93.8)
- added C64: 100nF/10V, Capacitor_SMD:C_0201_0603Metric, B.Cu at (85.6, 86.0)
- added C65: 100nF/10V, Capacitor_SMD:C_0201_0603Metric, B.Cu at (92.0, 85.9)
- added C66: 100nF/10V, Capacitor_SMD:C_0201_0603Metric, B.Cu at (85.2, 93.8)
- added C67: 10uF/6.4V, Capacitor_SMD:C_0402_1005Metric, B.Cu at (81.8, 84.9)
- added C68: 22uF/10V, Capacitor_SMD:C_0603_1608Metric, B.Cu at (91.7, 98.5)
- added C69: 1uF/10V, Capacitor_SMD:C_0402_1005Metric, B.Cu at (88.7, 98.4)
- added C7: 100nF/10V, Capacitor_SMD:C_0201_0603Metric, F.Cu at (86.5, 70.5)
- added C70: 100nF/10V, Capacitor_SMD:C_0201_0603Metric, B.Cu at (87.4, 95.0)
- added C71: 100nF/10V, Capacitor_SMD:C_0201_0603Metric, B.Cu at (84.9, 82.1)
- added C72: 100nF/10V, Capacitor_SMD:C_0201_0603Metric, B.Cu at (82.5, 90.5)
- added C73: 100nF/10V, Capacitor_SMD:C_0201_0603Metric, B.Cu at (82.6, 83.8)
- added C74: 100nF/10V, Capacitor_SMD:C_0201_0603Metric, B.Cu at (86.8, 88.0)
- added C75: 100nF/10V, Capacitor_SMD:C_0201_0603Metric, B.Cu at (82.5, 95.4)
- added C76: 100nF/10V, Capacitor_SMD:C_0201_0603Metric, B.Cu at (92.6, 95.0)
- added C77: 100nF/10V, Capacitor_SMD:C_0201_0603Metric, B.Cu at (82.5, 89.1)
- added C78: 100nF/10V, Capacitor_SMD:C_0201_0603Metric, B.Cu at (84.4, 83.4)
- added C79: 10uf/6.4V, Capacitor_SMD:C_0402_1005Metric, B.Cu at (89.8, 98.4)
- added C8: 100nF/10V, Capacitor_SMD:C_0201_0603Metric, F.Cu at (89.0, 69.0)
- added C80: 22uF/10V, Capacitor_SMD:C_0603_1608Metric, F.Cu at (118.0, 96.0)
- added C81: 1uF/10V, Capacitor_SMD:C_0402_1005Metric, F.Cu at (119.3, 95.4)
- added C82: 100nF/10V, Capacitor_SMD:C_0201_0603Metric, B.Cu at (122.2, 81.3)
- added C83: 100nF/10V, Capacitor_SMD:C_0201_0603Metric, B.Cu at (124.0, 78.3)
- added C84: 100nF/10V, Capacitor_SMD:C_0201_0603Metric, B.Cu at (127.2, 84.4)
- added C85: 100nF/10V, Capacitor_SMD:C_0201_0603Metric, B.Cu at (121.8, 84.3)
- added C86: 100nF/10V, Capacitor_SMD:C_0201_0603Metric, B.Cu at (122.4, 90.3)
- added C87: 100nF/10V, Capacitor_SMD:C_0201_0603Metric, F.Cu at (128.6, 91.5)
- added C88: 100nF/10V, Capacitor_SMD:C_0201_0603Metric, F.Cu at (128.0, 84.5)
- added C89: 100nF/10V, Capacitor_SMD:C_0201_0603Metric, B.Cu at (124.1, 94.0)
- added C9: 100nF/10V, Capacitor_SMD:C_0201_0603Metric, F.Cu at (86.5, 72.0)
- added C90: 100nF/10V, Capacitor_SMD:C_0201_0603Metric, B.Cu at (122.3, 91.3)
- added C91: 10uF/6.3V, Capacitor_SMD:C_0402_1005Metric, F.Cu at (120.5, 95.4)
- added C92: 10uF/6.3V, Capacitor_SMD:C_0402_1005Metric, B.Cu at (128.1, 81.8)
- added C93: 100nF/10V, Capacitor_SMD:C_0201_0603Metric, B.Cu at (116.4, 90.7)
- added C94: 100nF/10V, Capacitor_SMD:C_0201_0603Metric, B.Cu at (123.5, 82.6)
- added C95: 100nF/10V, Capacitor_SMD:C_0201_0603Metric, B.Cu at (120.7, 89.7)
- added C96: 100nF/10V, Capacitor_SMD:C_0201_0603Metric, B.Cu at (127.3, 82.1)
- added C97: 100nF/10V, Capacitor_SMD:C_0201_0603Metric, B.Cu at (117.5, 83.2)
- added C98: 100nF/10V, Capacitor_SMD:C_0201_0603Metric, F.Cu at (128.6, 90.5)
- added C99: 10uF/6.3V, Capacitor_SMD:C_0402_1005Metric, F.Cu at (128.8, 89.4)
- added D1: D_TVS, Diode_SMD:D_0402_1005Metric_Pad0.77x0.64mm_HandSolder, F.Cu at (79.4, 104.1)
- added D2: D_TVS, Diode_SMD:D_0402_1005Metric_Pad0.77x0.64mm_HandSolder, F.Cu at (77.2, 104.1)
- added D27: PCMF2USB3S, BeagleV:PCMF2USB3S, F.Cu at (80.5, 94.8)
- added D28: PCMF2USB3S, BeagleV:PCMF2USB3S, F.Cu at (80.5, 96.9)
- added D29: PCMF2USB3S, BeagleV:PCMF2USB3S, F.Cu at (80.5, 92.7)
- added D30: PCMF2USB3S, BeagleV:PCMF2USB3S, F.Cu at (80.6, 75.2)
- added D31: PCMF2USB3S, BeagleV:PCMF2USB3S, F.Cu at (80.6, 77.6)
- added D32: PCMF2USB3S, BeagleV:PCMF2USB3S, F.Cu at (80.6, 72.7)
- added D35: PMEG3010CEJ, Diode_SMD:D_SOD-323F, F.Cu at (94.0, 108.5)
- added D4: D_TVS, Diode_SMD:D_0402_1005Metric_Pad0.77x0.64mm_HandSolder, F.Cu at (116.2, 59.0)
- added D5: ESDPSA0402V05, Diode_SMD:D_0402_1005Metric_Pad0.77x0.64mm_HandSolder, B.Cu at (127.4, 49.2)
- added D52: SMBJ5.0CA-TR, Diode_SMD:D_SMB, F.Cu at (137.2, 57.9)
- added D6: PMEG3010CEJ, Diode_SMD:D_SOD-323F, B.Cu at (97.9, 53.8)
- added D62: Protection-Diode, Package_SON:USON-10_2.5x1.0mm_P0.5mm, B.Cu at (111.6, 56.2)
- added D63: Protection-Diode, Package_SON:USON-10_2.5x1.0mm_P0.5mm, B.Cu at (115.3, 56.2)
- added D64: Protection-Diode, Package_SON:USON-10_2.5x1.0mm_P0.5mm, F.Cu at (119.3, 59.3)
- added D65: PMEG3010CEJ, Diode_SMD:D_SOD-323F, B.Cu at (142.9, 54.8)
- added D7: PMEG3010CEJ, Diode_SMD:D_SOD-323F, B.Cu at (97.0, 64.5)
- added F2: Fuse, Fuse:Fuse_0603_1608Metric_Pad1.05x0.95mm_HandSolder, B.Cu at (121.6, 60.0)
- added FB1: FerriteBead, Inductor_SMD:L_0402_1005Metric_Pad0.77x0.64mm_HandSolder, B.Cu at (115.7, 61.9)
- added FB2: FerriteBead, Inductor_SMD:L_0402_1005Metric_Pad0.77x0.64mm_HandSolder, F.Cu at (115.2, 68.8)
- added FB3: FerriteBead, Inductor_SMD:L_0402_1005Metric_Pad0.77x0.64mm_HandSolder, B.Cu at (106.2, 62.4)
- added FB4: FerriteBead 120R, Inductor_SMD:L_0402_1005Metric_Pad0.77x0.64mm_HandSolder, F.Cu at (84.9, 75.5)
- added FB6: FerriteBead, Inductor_SMD:L_0402_1005Metric_Pad0.77x0.64mm_HandSolder, B.Cu at (82.7, 100.8)
- added FB7: FerriteBead 120R, Inductor_SMD:L_0402_1005Metric_Pad0.77x0.64mm_HandSolder, B.Cu at (106.0, 87.6)
- added FB8: FerriteBead 120R, Inductor_SMD:L_0402_1005Metric_Pad0.77x0.64mm_HandSolder, B.Cu at (106.8, 82.9)
- added FB9: FerriteBead 120R, Inductor_SMD:L_0402_1005Metric_Pad0.77x0.64mm_HandSolder, B.Cu at (131.2, 97.7)
- added G***: LOGO, LOGO, F.Cu at (110.5, 107.5)
- added G***: LOGO, LOGO, F.Cu at (98.6, 75.3)
- added J1: FPC_CONN_2X15P, BeagleV:FPC-1-1734248-5, F.Cu at (99.2, 59.7)
- added J10: MICRO_SD_ST_TF_003A_16_1x14_5mm, BeagleV:ST-TF-003A, B.Cu at (132.6, 81.2)
- added J11: ST-HD-010, BeagleV:HDMI-Type-A, F.Cu at (114.7, 45.5)
- added J12: JTAG-Connector, Connector:Tag-Connect_TC2050-IDC-NL_2x05_P1.27mm_Vertical, F.Cu at (69.1, 114.4)
- added J13: USB_TYPE_C, BeagleV:USB-Type-C, F.Cu at (136.8, 52.9)
- added J14: DNP Conn_01x03_Male, Connector_PinHeader_2.54mm:PinHeader_1x03_P2.54mm_Vertical, F.Cu at (104.3, 48.7)
- added J2: FPC_CONN_2X15P, BeagleV:FPC-1-1734248-5, F.Cu at (92.8, 59.8)
- added J3: audio_5p_mj2135_5d6_14_7x7x6mm, BeagleV:PJ322, F.Cu at (62.8, 107.2)
- added J4: USB-TYPE-A-3.0, BeagleV:Stacked-USB-TypeA, F.Cu at (61.9, 93.5)
- added J5: USB-TYPE-A-3.0, BeagleV:Stacked-USB-TypeA, F.Cu at (61.9, 75.8)
- added J6: LPJG0801HBNL, BeagleV:LPJG0801EBNL, F.Cu at (70.2, 56.8)
- added J7: PI-Connector-2x20-2.54mm, Connector_PinHeader_2.54mm:PinHeader_2x20_P2.54mm_Vertical, F.Cu at (139.8, 112.0)
- added J8: U.FL-R-SMT-1, BeagleV:U.FL-R-SMT-1, F.Cu at (144.1, 108.5)
- added J9: FPC_CONN_2X15P, BeagleV:FPC-1-1734248-5, F.Cu at (143.6, 84.5)
- added L1: 1uH, BeagleV:WPN201610H_2x1.6, F.Cu at (132.2, 58.5)
- added L2: 3.3uH, BeagleV:Sunlord_3.0x3.0, F.Cu at (132.7, 94.2)
- added L3: 10nH, Inductor_SMD:L_0201_0603Metric_Pad0.64x0.40mm_HandSolder, F.Cu at (146.2, 104.8)
- added L4: 0.47uH, BeagleV:Codaca_4.4x4.4, F.Cu at (122.4, 66.8)
- added L5: 0.56uH, BeagleV:Codaca_4.4x4.4, F.Cu at (137.2, 69.0)
- added L6: 10uH, Inductor_SMD:L_0805_2012Metric_Pad1.05x1.20mm_HandSolder, B.Cu at (139.2, 55.6)
- added L7: 1uH, BeagleV:WPN201610H_2x1.6, F.Cu at (136.3, 62.9)
- added L8: 1uH, BeagleV:WPN201610H_2x1.6, F.Cu at (129.0, 58.5)
- added LED1: GREEN LED, LED_SMD:LED_0603_1608Metric_Pad1.05x0.95mm_HandSolder, F.Cu at (144.8, 57.1)
- added LED2: RED LED, LED_SMD:LED_0603_1608Metric_Pad1.05x0.95mm_HandSolder, F.Cu at (144.7, 54.6)
- added OSC1: 32.768kHz-clock, BeagleV:7XZ-32.768KHz, F.Cu at (121.4, 99.5)
- added Q1: CJ1012, Package_TO_SOT_SMD:SOT-523, F.Cu at (144.3, 61.8)
- added Q2: CJ1012, Package_TO_SOT_SMD:SOT-523, B.Cu at (67.1, 78.8)
- added Q3: CJ1012, Package_TO_SOT_SMD:SOT-523, B.Cu at (139.7, 67.4)
- added Q6: CSD87381P, BeagleV:CSD87381P, F.Cu at (141.3, 67.8)
- added Q7: CSD87381P, BeagleV:CSD87381P, F.Cu at (123.4, 61.5)
- added Q8: IRLML6401, Package_TO_SOT_SMD:SOT-23, F.Cu at (141.3, 56.3)
- added Q9: BCM857BS-7F-F, Package_TO_SOT_SMD:SOT-363_SC-70-6_Handsoldering, B.Cu at (144.4, 67.6)
- added R1: 10K, Resistor_SMD:R_0201_0603Metric, F.Cu at (128.9, 84.4)
- added R10: 33R, Resistor_SMD:R_0201_0603Metric, F.Cu at (108.3, 102.2)
- added R100: 10K, Resistor_SMD:R_0402_1005Metric, B.Cu at (139.5, 70.1)
- added R101: 4.7K, Resistor_SMD:R_0402_1005Metric, F.Cu at (137.4, 77.1)
- added R102: 33R, Resistor_SMD:R_0201_0603Metric, F.Cu at (136.4, 77.3)
- added R103: 33R, Resistor_SMD:R_0201_0603Metric, F.Cu at (135.7, 77.3)
- added R104: 33R, Resistor_SMD:R_0201_0603Metric, F.Cu at (136.2, 87.2)
- added R105: 33R, Resistor_SMD:R_0201_0603Metric, F.Cu at (134.8, 77.3)
- added R106: 33R, Resistor_SMD:R_0201_0603Metric, F.Cu at (135.3, 87.2)
- added R107: 33R, Resistor_SMD:R_0201_0603Metric, F.Cu at (134.5, 87.2)
- added R108: 33R, Resistor_SMD:R_0201_0603Metric, F.Cu at (114.5, 100.5)
- added R109: 33R, Resistor_SMD:R_0201_0603Metric, F.Cu at (107.6, 102.2)
- added R11: 33R, Resistor_SMD:R_0201_0603Metric, F.Cu at (105.5, 102.2)
- added R110: 33R, Resistor_SMD:R_0201_0603Metric, F.Cu at (99.2, 100.5)
- added R111: 10K, Resistor_SMD:R_0402_1005Metric, F.Cu at (94.0, 106.5)
- added R112: 10K, Resistor_SMD:R_0402_1005Metric, F.Cu at (90.0, 99.9)
- added R113: 33R, Resistor_SMD:R_0201_0603Metric, F.Cu at (102.5, 100.5)
- added R114: 33R, Resistor_SMD:R_0201_0603Metric, F.Cu at (124.7, 98.3)
- added R115: 1M, Resistor_SMD:R_0402_1005Metric, B.Cu at (107.7, 76.5)
- added R116: 0R, Resistor_SMD:R_0402_1005Metric, B.Cu at (109.6, 76.5)
- added R117: 1K, Resistor_SMD:R_0402_1005Metric, F.Cu at (134.0, 58.7)
- added R118: 10K, Resistor_SMD:R_0402_1005Metric, B.Cu at (127.2, 50.2)
- added R119: 0R, Resistor_SMD:R_0402_1005Metric, B.Cu at (124.6, 70.0)
- added R12: 33R, Resistor_SMD:R_0201_0603Metric, F.Cu at (106.9, 100.5)
- added R120: 1M, Resistor_SMD:R_0402_1005Metric, F.Cu at (103.5, 76.9)
- added R121: 0R, Resistor_SMD:R_0402_1005Metric, B.Cu at (124.6, 71.0)
- added R122: 0R, Resistor_SMD:R_0402_1005Metric, F.Cu at (105.8, 76.9)
- added R123: 10K, Resistor_SMD:R_0201_0603Metric, F.Cu at (129.7, 84.4)
- added R124: 10K, Resistor_SMD:R_0201_0603Metric, F.Cu at (130.5, 84.4)
- added R125: 10K, Resistor_SMD:R_0201_0603Metric, F.Cu at (104.8, 102.2)
- added R126: 10K, Resistor_SMD:R_0201_0603Metric, F.Cu at (131.9, 77.8)
- added R127: 4.7K, Resistor_SMD:R_0402_1005Metric, B.Cu at (100.4, 53.7)
- added R128: 4.7K, Resistor_SMD:R_0402_1005Metric, B.Cu at (100.4, 54.7)
- added R129: 4.7K, Resistor_SMD:R_0402_1005Metric, B.Cu at (94.0, 53.9)
- added R13: 33R, Resistor_SMD:R_0201_0603Metric, F.Cu at (109.0, 100.5)
- added R130: DNP, Resistor_SMD:R_0201_0603Metric, B.Cu at (129.9, 106.9)
- added R131: 4.7K, Resistor_SMD:R_0402_1005Metric, B.Cu at (94.0, 54.8)
- added R133: 0R, Resistor_SMD:R_0201_0603Metric, F.Cu at (143.0, 104.3)
- added R134: 10K, Resistor_SMD:R_0201_0603Metric, F.Cu at (131.9, 77.0)
- added R135: DNP, Resistor_SMD:R_0201_0603Metric, F.Cu at (142.6, 104.6)
- added R136: DNP, Resistor_SMD:R_0402_1005Metric, B.Cu at (129.9, 104.3)
- added R137: 10K, Resistor_SMD:R_0201_0603Metric, F.Cu at (124.7, 99.2)
- added R138: 10K, Resistor_SMD:R_0402_1005Metric, B.Cu at (65.5, 78.9)
- added R139: DNP, Resistor_SMD:R_0402_1005Metric, B.Cu at (138.1, 97.6)
- added R14: 33R, Resistor_SMD:R_0201_0603Metric, F.Cu at (106.9, 102.2)
- added R140: 0R, Resistor_SMD:R_0402_1005Metric, B.Cu at (137.1, 97.6)
- added R141: DNP, Resistor_SMD:R_0201_0603Metric, B.Cu at (136.0, 97.8)
- added R142: 10K, Resistor_SMD:R_0402_1005Metric, F.Cu at (132.1, 70.8)
- added R143: 1M, Resistor_SMD:R_0402_1005Metric, B.Cu at (94.4, 69.6)
- added R144: 100K, Resistor_SMD:R_0402_1005Metric, B.Cu at (89.1, 65.4)
- added R145: 33R, Resistor_SMD:R_0201_0603Metric, B.Cu at (103.5, 100.8)
- added R146: 100K, Resistor_SMD:R_0402_1005Metric, F.Cu at (89.1, 65.4)
- added R147: 10K, Resistor_SMD:R_0201_0603Metric, F.Cu at (131.8, 76.2)
- added R148: 10K, Resistor_SMD:R_0201_0603Metric, B.Cu at (135.3, 97.8)
- added R149: 10K, Resistor_SMD:R_0201_0603Metric, B.Cu at (134.6, 97.8)
- added R15: 33R, Resistor_SMD:R_0201_0603Metric, F.Cu at (110.4, 100.5)
- added R150: 10K, Resistor_SMD:R_0201_0603Metric, B.Cu at (133.9, 97.8)
- added R151: 1M, Resistor_SMD:R_1206_3216Metric, B.Cu at (90.6, 50.8)
- added R152: 10K, Resistor_SMD:R_0201_0603Metric, B.Cu at (133.0, 97.8)
- added R153: 10K, Resistor_SMD:R_0201_0603Metric, B.Cu at (132.1, 97.8)
- added R154: DNP, Resistor_SMD:R_0402_1005Metric, F.Cu at (138.0, 94.9)
- added R155: 0R, Resistor_SMD:R_0402_1005Metric, F.Cu at (136.8, 93.9)
- added R156: 33R, Resistor_SMD:R_0201_0603Metric, F.Cu at (101.7, 100.5)
- added R157: 33R, Resistor_SMD:R_0201_0603Metric, B.Cu at (101.8, 100.8)
- added R158: 33R, Resistor_SMD:R_0201_0603Metric, B.Cu at (102.7, 100.8)
- added R159: 10k, Resistor_SMD:R_0402_1005Metric, F.Cu at (144.3, 63.9)
- added R16: 33R, Resistor_SMD:R_0201_0603Metric, F.Cu at (110.4, 102.2)
- added R160: 100K, Resistor_SMD:R_0402_1005Metric, B.Cu at (128.4, 106.5)
- added R161: 1K, Resistor_SMD:R_0402_1005Metric, B.Cu at (96.2, 53.7)
- added R162: 49.9K, Resistor_SMD:R_0402_1005Metric, B.Cu at (145.0, 71.6)
- added R163: 49.9K, Resistor_SMD:R_0402_1005Metric, B.Cu at (143.8, 71.6)
- added R164: DNP, Resistor_SMD:R_0402_1005Metric, F.Cu at (118.7, 67.7)
- added R165: 0R, Resistor_SMD:R_0402_1005Metric, B.Cu at (91.6, 62.8)
- added R166: 0R, Resistor_SMD:R_0402_1005Metric, B.Cu at (125.8, 58.4)
- added R167: 4.7K, Resistor_SMD:R_0402_1005Metric, B.Cu at (139.5, 69.0)
- added R17: 33R, Resistor_SMD:R_0201_0603Metric, F.Cu at (109.7, 102.2)
- added R18: 33R, Resistor_SMD:R_0201_0603Metric, F.Cu at (105.5, 100.5)
- added R184: 240R, Resistor_SMD:R_0402_1005Metric, F.Cu at (88.9, 81.3)
- added R19: 33R, Resistor_SMD:R_0201_0603Metric, F.Cu at (113.9, 100.5)
- added R2: 1K, Resistor_SMD:R_0402_1005Metric, F.Cu at (141.5, 63.3)
- added R20: 33R, Resistor_SMD:R_0201_0603Metric, F.Cu at (111.1, 102.2)
- added R21: 33R, Resistor_SMD:R_0201_0603Metric, F.Cu at (106.2, 102.2)
- added R22: 33R, Resistor_SMD:R_0201_0603Metric, F.Cu at (113.9, 102.3)
- added R23: 680R, Resistor_SMD:R_0402_1005Metric, B.Cu at (94.2, 65.2)
- added R232: 33R, Resistor_SMD:R_0201_0603Metric, F.Cu at (133.4, 76.2)
- added R233: 33R, Resistor_SMD:R_0201_0603Metric, F.Cu at (133.3, 77.0)
- added R234: 33R, Resistor_SMD:R_0201_0603Metric, F.Cu at (133.3, 77.8)
- added R235: 33R, Resistor_SMD:R_0201_0603Metric, F.Cu at (104.8, 100.5)
- added R236: 33R, Resistor_SMD:R_0201_0603Metric, F.Cu at (130.5, 86.3)
- added R237: 33R, Resistor_SMD:R_0201_0603Metric, F.Cu at (129.7, 86.3)
- added R238: 33R, Resistor_SMD:R_0201_0603Metric, F.Cu at (128.9, 86.3)
- added R24: 27K, Resistor_SMD:R_0402_1005Metric, B.Cu at (69.0, 76.7)
- added R240: DNP, Resistor_SMD:R_0402_1005Metric, F.Cu at (86.1, 78.1)
- added R241: 10K, Resistor_SMD:R_0402_1005Metric, F.Cu at (85.1, 78.1)
- added R242: DNP, Resistor_SMD:R_0402_1005Metric, F.Cu at (89.0, 78.1)
- added R243: 10K, Resistor_SMD:R_0402_1005Metric, F.Cu at (90.0, 78.1)
- added R244: DNP, Resistor_SMD:R_0402_1005Metric, F.Cu at (87.0, 78.1)
- added R245: 10K, Resistor_SMD:R_0402_1005Metric, F.Cu at (88.0, 78.1)
- added R246: 10K, Resistor_SMD:R_0402_1005Metric, B.Cu at (95.1, 78.2)
- added R247: DNP, Resistor_SMD:R_0402_1005Metric, B.Cu at (94.1, 78.2)
- added R248: 5.1K, Resistor_SMD:R_0402_1005Metric, F.Cu at (134.5, 55.6)
- added R249: 5.1K, Resistor_SMD:R_0402_1005Metric, F.Cu at (133.6, 55.6)
- added R25: 100K, Resistor_SMD:R_0402_1005Metric, B.Cu at (90.3, 65.4)
- added R252: 10K, Resistor_SMD:R_0402_1005Metric, B.Cu at (124.9, 58.4)
- added R254: 0R, Resistor_SMD:R_0402_1005Metric, F.Cu at (144.3, 67.2)
- added R255: 0R, Resistor_SMD:R_0402_1005Metric, F.Cu at (144.3, 68.3)
- added R256: 12.1K, Resistor_SMD:R_0402_1005Metric, F.Cu at (133.6, 70.8)
- added R257: 0R, Resistor_SMD:R_0402_1005Metric, B.Cu at (124.2, 64.3)
- added R258: 2.2K, Resistor_SMD:R_0402_1005Metric, F.Cu at (126.8, 59.1)
- added R259: 0R, Resistor_SMD:R_0402_1005Metric, F.Cu at (120.0, 62.2)
- added R26: 100K, Resistor_SMD:R_0402_1005Metric, F.Cu at (84.8, 72.4)
- added R260: 0R, Resistor_SMD:R_0402_1005Metric, F.Cu at (120.0, 63.3)
- added R261: 49.9K, Resistor_SMD:R_0402_1005Metric, B.Cu at (144.3, 61.2)
- added R262: 12.1K, Resistor_SMD:R_0402_1005Metric, B.Cu at (125.8, 68.0)
- added R263: 1M, Resistor_SMD:R_0402_1005Metric, B.Cu at (137.4, 61.4)
- added R264: 13.3K, Resistor_SMD:R_0402_1005Metric, B.Cu at (142.2, 61.7)
- added R265: 33R, Resistor_SMD:R_0201_0603Metric, F.Cu at (77.9, 112.8)
- added R266: 33R, Resistor_SMD:R_0201_0603Metric, F.Cu at (77.8, 114.0)
- added R267: 33R, Resistor_SMD:R_0201_0603Metric, F.Cu at (78.8, 106.6)
- added R268: 33R, Resistor_SMD:R_0201_0603Metric, F.Cu at (78.0, 106.6)
- added R269: 120R, Resistor_SMD:R_0402_1005Metric, F.Cu at (80.1, 112.8)
- added R27: 0R, Resistor_SMD:R_0402_1005Metric, B.Cu at (114.8, 68.2)
- added R270: 120R, Resistor_SMD:R_0402_1005Metric, F.Cu at (78.9, 108.7)
- added R271: 120R, Resistor_SMD:R_0402_1005Metric, F.Cu at (80.1, 114.1)
- added R272: 120R, Resistor_SMD:R_0402_1005Metric, F.Cu at (77.8, 108.7)
- added R28: 10K, Resistor_SMD:R_0201_0603Metric, F.Cu at (112.1, 72.1)
- added R29: 10K, Resistor_SMD:R_0201_0603Metric, F.Cu at (82.7, 51.7)
- added R3: 1K, Resistor_SMD:R_0402_1005Metric, F.Cu at (140.5, 63.3)
- added R30: 10K, Resistor_SMD:R_0201_0603Metric, F.Cu at (82.7, 52.6)
- added R31: 10K, Resistor_SMD:R_0201_0603Metric, F.Cu at (107.5, 72.0)
- added R32: 10K, Resistor_SMD:R_0201_0603Metric, F.Cu at (108.7, 72.0)
- added R33: 10K, Resistor_SMD:R_0201_0603Metric, F.Cu at (109.9, 72.0)
- added R34: 10K, Resistor_SMD:R_0201_0603Metric, F.Cu at (111.0, 72.1)
- added R35: 1K, Resistor_SMD:R_0402_1005Metric, F.Cu at (114.3, 72.1)
- added R36: 1K, Resistor_SMD:R_0201_0603Metric, F.Cu at (113.3, 72.1)
- added R37: 0R, Resistor_SMD:R_0402_1005Metric, B.Cu at (108.3, 62.9)
- added R38: 1K, Resistor_SMD:R_0402_1005Metric, F.Cu at (111.4, 74.7)
- added R39: 1K, Resistor_SMD:R_0201_0603Metric, F.Cu at (115.2, 70.0)
- added R4: 4.7K, Resistor_SMD:R_0402_1005Metric, F.Cu at (142.5, 63.3)
- added R41: 33R, Resistor_SMD:R_0201_0603Metric, B.Cu at (100.4, 76.6)
- added R42: 33R, Resistor_SMD:R_0201_0603Metric, B.Cu at (104.0, 76.6)
- added R43: 33R, Resistor_SMD:R_0201_0603Metric, B.Cu at (105.6, 76.5)
- added R44: 33R, Resistor_SMD:R_0201_0603Metric, B.Cu at (101.3, 76.6)
- added R45: 33R, Resistor_SMD:R_0201_0603Metric, B.Cu at (102.2, 76.6)
- added R46: 33R, Resistor_SMD:R_0201_0603Metric, B.Cu at (98.2, 76.6)
- added R47: 33R, Resistor_SMD:R_0201_0603Metric, F.Cu at (112.5, 74.3)
- added R48: 33R, Resistor_SMD:R_0201_0603Metric, F.Cu at (111.4, 76.8)
- added R49: 33R, Resistor_SMD:R_0201_0603Metric, F.Cu at (110.4, 74.4)
- added R5: 33R, Resistor_SMD:R_0201_0603Metric, F.Cu at (109.7, 100.5)
- added R50: 33R, Resistor_SMD:R_0201_0603Metric, F.Cu at (109.5, 74.4)
- added R51: 33R, Resistor_SMD:R_0201_0603Metric, F.Cu at (108.7, 74.4)
- added R52: 33R, Resistor_SMD:R_0201_0603Metric, F.Cu at (107.5, 74.4)
- added R53: 33R, Resistor_SMD:R_0201_0603Metric, F.Cu at (113.3, 74.3)
- added R54: 33R, Resistor_SMD:R_0201_0603Metric, F.Cu at (114.2, 74.3)
- added R55: 1K, Resistor_SMD:R_0402_1005Metric, F.Cu at (82.2, 55.8)
- added R56: 1K, Resistor_SMD:R_0402_1005Metric, F.Cu at (82.2, 56.9)
- added R57: 1M, Resistor_SMD:R_0402_1005Metric, F.Cu at (114.8, 63.2)
- added R58: 0R, Resistor_SMD:R_0402_1005Metric, F.Cu at (119.3, 65.8)
- added R59: 0R, Resistor_SMD:R_0402_1005Metric, F.Cu at (91.9, 78.1)
- added R6: 33R, Resistor_SMD:R_0201_0603Metric, F.Cu at (108.3, 100.5)
- added R60: 12K, Resistor_SMD:R_0402_1005Metric, B.Cu at (112.2, 63.5)
- added R61: DNP, Resistor_SMD:R_0402_1005Metric, F.Cu at (82.9, 54.1)
- added R62: 240R, Resistor_SMD:R_0402_1005Metric, F.Cu at (86.4, 81.2)
- added R63: 0R, Resistor_SMD:R_0402_1005Metric, F.Cu at (136.3, 65.6)
- added R64: 10K, Resistor_SMD:R_0402_1005Metric, F.Cu at (81.2, 86.3)
- added R65: DNP, Resistor_SMD:R_0402_1005Metric, F.Cu at (81.2, 84.3)
- added R66: DNP, Resistor_SMD:R_0402_1005Metric, F.Cu at (81.2, 85.3)
- added R67: 0R, Resistor_SMD:R_0402_1005Metric, F.Cu at (81.2, 87.3)
- added R68: 10K, Resistor_SMD:R_0402_1005Metric, F.Cu at (81.2, 90.3)
- added R69: DNP, Resistor_SMD:R_0402_1005Metric, F.Cu at (81.2, 88.3)
- added R7: 33R, Resistor_SMD:R_0201_0603Metric, F.Cu at (111.8, 100.5)
- added R70: DNP, Resistor_SMD:R_0402_1005Metric, F.Cu at (81.2, 89.3)
- added R71: 240R, Resistor_SMD:R_0402_1005Metric, F.Cu at (120.8, 76.6)
- added R72: 240R, Resistor_SMD:R_0402_1005Metric, F.Cu at (123.1, 76.6)
- added R73: 10K, Resistor_SMD:R_0402_1005Metric, B.Cu at (115.8, 85.8)
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Other:
- board outline added: 85.1 x 70.2 mm
- copper layers 0 -> 12
- board text added: "BeagleV - StartLight"
