File: BeagleV/BeagleV.kicad_pcb (KiCad board)
At the start: 12 copper layers, 85.1 x 70.2 mm, 576 parts, among them J1 FPC_CONN_2X15P, J10 MICRO_SD_ST_TF_003A_16_1x14_5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, J11 ST-HD-010, J12 JTAG-Connector, J13 USB_TYPE_C, J14 DNP Conn_01x03_Male, J2 FPC_CONN_2X15P, J3 audio_5p_mj2135_5d6_14_7x7x6mm, J4 USB-TYPE-A-3.0, J5 USB-TYPE-A-3.0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

Commit message: Display and camera connector footprint updated
Parts:
- moved J9 0.50 mm to (143.1, 84.5), turned to 180 degrees
