File: BeagleV/BeagleV_CSI_Conn.kicad_sch (KiCad schematic)
At the start: 4 parts, among them J1 FPC_CONN_2X15P, j2 FPC_CONN_2X15P

Commit message: Initial commit to working branch, Cloned from the gitlab repository
Parts:
- C1: footprint (none) -> Capacitor_SMD:C_0201_0603Metric
- C2: renamed from C100nF/10V; value C_Small -> 100nF/10V1; footprint (none) -> Capacitor_SMD:C_0201_0603Metric
- J1: footprint (none) -> BeagleV:FPC-1-1734248-5
- J2: renamed from j2; footprint (none) -> BeagleV:FPC-1-1734248-5
Changed lines of the file:
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@@
   (title_block
     (title "Beagle V")
-    (date "2021-06-03")
+    (date "2021-06-11")
     (rev "v0.7")
   )
@@
       (effects (font (size 1.27 1.27)) (justify left))
     )
-    (property "Footprint" "" (id 2) (at 229.87 130.81 0)
+    (property "Footprint" "Capacitor_SMD:C_0201_0603Metric" (id 2) (at 229.87 130.81 0)
       (effects (font (size 1.27 1.27)) hide)
     )
@@
   (symbol (lib_id "Device:C_Small") (at 229.87 209.55 0) (unit 1)
     (in_bom yes) (on_board yes) (fields_autoplaced)
-    (property "Reference" "C100nF/10V" (id 0) (at 232.1942 208.7891 0)
+    (property "Reference" "C2" (id 0) (at 232.1942 208.7891 0)
       (effects (font (size 1.27 1.27)) (justify left))
     )
-    (property "Value" "C_Small" (id 1) (at 232.1942 211.0878 0)
+    (property "Value" "100nF/10V1" (id 1) (at 232.1942 211.0878 0)
       (effects (font (size 1.27 1.27)) (justify left))
     )
-    (property "Footprint" "" (id 2) (at 229.87 209.55 0)
+    (property "Footprint" "Capacitor_SMD:C_0201_0603Metric" (id 2) (at 229.87 209.55 0)
       (effects (font (size 1.27 1.27)) hide)
     )
@@
     (property "Reference" "J1" (id 0) (at 266.7 75.3576 0))
     (property "Value" "FPC_CONN_2X15P" (id 1) (at 266.7 77.6563 0))
-    (property "Footprint" "" (id 2) (at 263.398 92.329 0)
+    (property "Footprint" "BeagleV:FPC-1-1734248-5" (id 2) (at 263.398 92.329 0)
       (effects (font (size 1.27 1.27)) hide)
     )
@@
   (symbol (lib_id "BeagleV:FPC_CONN_2X15P") (at 266.7 179.07 0) (unit 1)
     (in_bom yes) (on_board yes) (fields_autoplaced)
-    (property "Reference" "j2" (id 0) (at 266.7 154.0976 0))
+    (property "Reference" "J2" (id 0) (at 266.7 154.0976 0))
     (property "Value" "FPC_CONN_2X15P" (id 1) (at 266.7 156.3963 0))
-    (property "Footprint" "" (id 2) (at 263.398 171.069 0)
-      (effects (font (size 1.27 1.27)) hide)
-    )
+    (property "Footprint" "BeagleV:FPC-1-1734248-5" (id 2) (at 263.398 171.069 0)
+      (effects (font (size 1.27 1.27)) hide)
+    )
