File: BeagleV/BeagleV_DSI_Audio.kicad_sch (KiCad schematic)
At the start: 21 parts, among them J3 audio_5p_mj2135_5d6_14_7x7x6mm, J9 FPC_CONN_2X15P

Commit message: Initial commit to working branch, Cloned from the gitlab repository
Parts:
- C272: footprint (none) -> Capacitor_SMD:C_0201_0603Metric
- C309, C310, C311, C312, C313, C314: footprint (none) -> Capacitor_SMD:C_0402_1005Metric
- D1, D2: footprint (none) -> Diode_SMD:D_0402_1005Metric_Pad0.77x0.64mm_HandSolder
- J3: footprint (none) -> BeagleV:PJ322
- J9: footprint (none) -> BeagleV:FPC-1-1734248-5
- R265, R266, R267, R268: footprint (none) -> Resistor_SMD:R_0201_0603Metric
- R269, R270, R271, R272: footprint (none) -> Resistor_SMD:R_0402_1005Metric
Changed lines of the file:
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@@
   (title_block
     (title "Beagle V")
-    (date "2021-06-03")
+    (date "2021-06-11")
     (rev "v0.7")
   )
@@
     (property "Reference" "R269" (id 0) (at 167.64 186.3302 90))
     (property "Value" "120R" (id 1) (at 167.64 188.6289 90))
-    (property "Footprint" "" (id 2) (at 167.64 190.5 0)
+    (property "Footprint" "Resistor_SMD:R_0402_1005Metric" (id 2) (at 167.64 190.5 0)
       (effects (font (size 1.27 1.27)) hide)
     )
@@
     (property "Reference" "R271" (id 0) (at 167.64 201.5702 90))
     (property "Value" "120R" (id 1) (at 167.64 203.8689 90))
-    (property "Footprint" "" (id 2) (at 167.64 205.74 0)
+    (property "Footprint" "Resistor_SMD:R_0402_1005Metric" (id 2) (at 167.64 205.74 0)
       (effects (font (size 1.27 1.27)) hide)
     )
@@
     (property "Reference" "R265" (id 0) (at 179.07 186.3302 90))
     (property "Value" "33R" (id 1) (at 179.07 188.6289 90))
-    (property "Footprint" "" (id 2) (at 179.07 190.5 0)
+    (property "Footprint" "Resistor_SMD:R_0201_0603Metric" (id 2) (at 179.07 190.5 0)
       (effects (font (size 1.27 1.27)) hide)
     )
@@
     (property "Reference" "R266" (id 0) (at 179.07 201.5702 90))
     (property "Value" "33R" (id 1) (at 179.07 203.8689 90))
-    (property "Footprint" "" (id 2) (at 179.07 205.74 0)
+    (property "Footprint" "Resistor_SMD:R_0201_0603Metric" (id 2) (at 179.07 205.74 0)
       (effects (font (size 1.27 1.27)) hide)
     )
@@
     (property "Reference" "R270" (id 0) (at 198.12 186.3302 90))
     (property "Value" "120R" (id 1) (at 198.12 188.6289 90))
-    (property "Footprint" "" (id 2) (at 198.12 190.5 0)
+    (property "Footprint" "Resistor_SMD:R_0402_1005Metric" (id 2) (at 198.12 190.5 0)
       (effects (font (size 1.27 1.27)) hide)
     )
@@
     (property "Reference" "R272" (id 0) (at 198.12 201.5702 90))
     (property "Value" "120R" (id 1) (at 198.12 203.8689 90))
-    (property "Footprint" "" (id 2) (at 198.12 205.74 0)
+    (property "Footprint" "Resistor_SMD:R_0402_1005Metric" (id 2) (at 198.12 205.74 0)
       (effects (font (size 1.27 1.27)) hide)
     )
@@
     (property "Reference" "R267" (id 0) (at 208.28 186.3302 90))
     (property "Value" "33R" (id 1) (at 208.28 188.6289 90))
-    (property "Footprint" "" (id 2) (at 208.28 190.5 0)
+    (property "Footprint" "Resistor_SMD:R_0201_0603Metric" (id 2) (at 208.28 190.5 0)
       (effects (font (size 1.27 1.27)) hide)
     )
@@
     (property "Reference" "R268" (id 0) (at 208.28 201.5702 90))
     (property "Value" "33R" (id 1) (at 208.28 203.8689 90))
-    (property "Footprint" "" (id 2) (at 208.28 205.74 0)
+    (property "Footprint" "Resistor_SMD:R_0201_0603Metric" (id 2) (at 208.28 205.74 0)
       (effects (font (size 1.27 1.27)) hide)
     )
@@
     (property "Reference" "C309" (id 0) (at 143.51 185.5047 90))
     (property "Value" "1uF/10V" (id 1) (at 143.51 187.8034 90))
-    (property "Footprint" "" (id 2) (at 143.51 190.5 0)
+    (property "Footprint" "Capacitor_SMD:C_0402_1005Metric" (id 2) (at 143.51 190.5 0)
       (effects (font (size 1.27 1.27)) hide)
     )
@@
     (property "Reference" "C310" (id 0) (at 143.51 200.7447 90))
     (property "Value" "1uF/10V" (id 1) (at 143.51 203.0434 90))
-    (property "Footprint" "" (id 2) (at 143.51 205.74 0)
+    (property "Footprint" "Capacitor_SMD:C_0402_1005Metric" (id 2) (at 143.51 205.74 0)
       (effects (font (size 1.27 1.27)) hide)
     )
@@
     (property "Reference" "C311" (id 0) (at 179.07 193.1247 90))
     (property "Value" "10nF/50V" (id 1) (at 179.07 195.4234 90))
-    (property "Footprint" "" (id 2) (at 179.07 198.12 0)
+    (property "Footprint" "Capacitor_SMD:C_0402_1005Metric" (id 2) (at 179.07 198.12 0)
       (effects (font (size 1.27 1.27)) hide)
     )
@@
     (property "Reference" "C313" (id 0) (at 179.07 208.3647 90))
     (property "Value" "10nF/50V" (id 1) (at 179.07 210.6634 90))
-    (property "Footprint" "" (id 2) (at 179.07 213.36 0)
+    (property "Footprint" "Capacitor_SMD:C_0402_1005Metric" (id 2) (at 179.07 213.36 0)
       (effects (font (size 1.27 1.27)) hide)
     )
@@
     (property "Reference" "C312" (id 0) (at 208.28 193.1247 90))
     (property "Value" "10nF/50V" (id 1) (at 208.28 195.4234 90))
-    (property "Footprint" "" (id 2) (at 208.28 198.12 0)
+    (property "Footprint" "Capacitor_SMD:C_0402_1005Metric" (id 2) (at 208.28 198.12 0)
       (effects (font (size 1.27 1.27)) hide)
     )
@@
     (property "Reference" "C314" (id 0) (at 208.28 208.3647 90))
     (property "Value" "10nF/50V" (id 1) (at 208.28 210.6634 90))
-    (property "Footprint" "" (id 2) (at 208.28 213.36 0)
+    (property "Footprint" "Capacitor_SMD:C_0402_1005Metric" (id 2) (at 208.28 213.36 0)
       (effects (font (size 1.27 1.27)) hide)
     )
@@
       (effects (font (size 1.27 1.27)) (justify left))
     )
-    (property "Footprint" "" (id 2) (at 226.06 127 0)
+    (property "Footprint" "Capacitor_SMD:C_0201_0603Metric" (id 2) (at 226.06 127 0)
       (effects (font (size 1.27 1.27)) hide)
     )
@@
       (effects (font (size 1.27 1.27)) (justify right))
     )
-    (property "Footprint" "" (id 2) (at 227.33 219.71 0)
+    (property "Footprint" "Diode_SMD:D_0402_1005Metric_Pad0.77x0.64mm_HandSolder" (id 2) (at 227.33 219.71 0)
       (effects (font (size 1.27 1.27)) hide)
     )
@@
       (effects (font (size 1.27 1.27)) (justify right))
     )
-    (property "Footprint" "" (id 2) (at 236.22 219.71 0)
+    (property "Footprint" "Diode_SMD:D_0402_1005Metric_Pad0.77x0.64mm_HandSolder" (id 2) (at 236.22 219.71 0)
       (effects (font (size 1.27 1.27)) hide)
     )
@@
       (effects (font (size 1.27 1.27)) (justify left))
     )
-    (property "Footprint" "" (id 2) (at 262.89 203.2 0)
+    (property "Footprint" "BeagleV:PJ322" (id 2) (at 262.89 203.2 0)
       (effects (font (size 1.27 1.27)) hide)
     )
@@
     (property "Reference" "J9" (id 0) (at 262.89 71.5476 0))
     (property "Value" "FPC_CONN_2X15P" (id 1) (at 262.89 73.8463 0))
-    (property "Footprint" "" (id 2) (at 259.588 88.519 0)
-      (effects (font (size 1.27 1.27)) hide)
-    )
+    (property "Footprint" "BeagleV:FPC-1-1734248-5" (id 2) (at 259.588 88.519 0)
+      (effects (font (size 1.27 1.27)) hide)
+    )
