File: BeagleV/BeagleV_Ethernet.kicad_sch (KiCad schematic)
At the start: 74 parts, among them J6 LPJG0801HBNL, U5 KSZ9031RNXCA, X6 25MHz - Crystal

Commit message: Initial commit to working branch, Cloned from the gitlab repository
Parts:
- removed P? (x2): VETH1_AVDDL_PLL, symbol BeagleV:VETH1_AVDDL_PLL
- removed P? (x7): VETH1_DVDDH, symbol BeagleV:VETH1_DVDDH
- removed P? (x5): VETH1_AVDDH, symbol BeagleV:VETH1_AVDDH
- C228: footprint (none) -> Capacitor_SMD:C_1206_3216Metric
- C28, C30, C31, C32, C34, C36, C38, C40, C42, C43, C45, C47: footprint (none) -> Capacitor_SMD:C_0402_1005Metric
- C29, C33, C35, C37, C39: footprint (none) -> Capacitor_SMD:C_0201_0603Metric
- FB1, FB2, FB3: footprint (none) -> Inductor_SMD:L_0402_1005Metric_Pad0.77x0.64mm_HandSolder
- J6: footprint (none) -> BeagleV:LPJG0801EBNL
- R151: footprint (none) -> Resistor_SMD:R_1206_3216Metric
- R164, R27, R35, R37, R38, R55, R56, R57, R58, R60, R61: footprint (none) -> Resistor_SMD:R_0402_1005Metric
- R28, R29, R30, R31, R32, R33, R34, R36, R39, R41, R42, R43, R44, R45, R46, R47, R48, R49, R50, R51, R52, R53, R54: footprint (none) -> Resistor_SMD:R_0201_0603Metric
- U5: footprint (none) -> BeagleV:KSZ9031RNX-QFN-48_EP_7.3x7.3_Pitch0.5mm
- X6: footprint (none) -> BeagleV:SMCE-2520
Connections:
- net GND: now also C31.2, C33.2
- net LDO_3V3 renamed VETH1_DVDDH
- net VETH1_DVDDH: no longer C31.1, C32.1, C33.1, C36.1, C37.1, C38.1, C39.1, C40.1, FB1.2, FB2.2, R37.2, R61.1, U5.1 (AVDDH_1), U5.12 (AVDDH_2), U5.4 (AVDDL_1), U5.44 (ADDL_PLL), U5.47 (AVDDH_3), U5.9 (AVDDL_2)
- new net VETH1_AVDDH: C31.1, C32.1, C33.1, C36.1, C37.1, FB1.2, R37.2, R61.1, U5.1 (AVDDH_1), U5.12 (AVDDH_2), U5.4 (AVDDL_1), U5.47 (AVDDH_3), U5.9 (AVDDL_2)
- new net VETH1_AVDDL_PLL: C38.1, C39.1, C40.1, FB2.2, U5.44 (ADDL_PLL)
