File: BeagleV/BeagleV_Hdmi_Framer.kicad_sch (KiCad schematic)
At the start: 23 parts, among them J11 ST-HD-010, U11 TDA19988

Commit message: Initial commit to working branch, Cloned from the gitlab repository
Parts:
- removed P?: HDMI_1V8, symbol BeagleV:HDMI_1V8
- C200, C266, C268, C271: footprint (none) -> Capacitor_SMD:C_0402_1005Metric
- C201, C267, C269, C270: footprint (none) -> Capacitor_SMD:C_0201_0603Metric
- D35: footprint (none) -> Diode_SMD:D_SOD-323F
- D4: footprint (none) -> Diode_SMD:D_0402_1005Metric_Pad0.77x0.64mm_HandSolder
- D62, D63, D64: footprint (none) -> Package_SON:USON-10_2.5x1.0mm_P0.5mm
- F2: footprint (none) -> Fuse:Fuse_0603_1608Metric_Pad1.05x0.95mm_HandSolder
- FB6: footprint (none) -> Inductor_SMD:L_0402_1005Metric_Pad0.77x0.64mm_HandSolder
- J11: footprint (none) -> BeagleV:HDMI-Type-A
- R111, R112, R84, R85, R86: footprint (none) -> Resistor_SMD:R_0402_1005Metric
- U11: footprint (none) -> BeagleV:TDA19988-QFN-64_EP_9x9_Pitch0.5mm
Connections:
- net LDO_3V3 renamed HDMI_1V8
Changed lines of the file:
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@@
   (title_block
     (title "Beagle V")
-    (date "2021-06-03")
+    (date "2021-06-11")
     (rev "v0.7")
   )
@@
   (symbol (lib_id "BeagleV:HDMI_1V8") (at 222.25 165.1 0) (unit 1)
     (in_bom yes) (on_board yes)
-    (property "Reference" "P?" (id 0) (at 222.25 165.1 0)
+    (property "Reference" "#P025" (id 0) (at 222.25 165.1 0)
       (effects (font (size 1.27 1.27)) hide)
     )
@@
       (effects (font (size 1.27 1.27)) (justify right))
     )
-    (property "Footprint" "" (id 2) (at 104.14 81.915 0)
+    (property "Footprint" "Resistor_SMD:R_0402_1005Metric" (id 2) (at 104.14 81.915 0)
       (effects (font (size 1.27 1.27)) hide)
     )
@@
       (effects (font (size 1.27 1.27)) (justify left))
     )
-    (property "Footprint" "" (id 2) (at 173.99 78.74 0)
+    (property "Footprint" "Resistor_SMD:R_0402_1005Metric" (id 2) (at 173.99 78.74 0)
       (effects (font (size 1.27 1.27)) hide)
     )
@@
     (property "Reference" "R111" (id 0) (at 175.895 157.7552 90))
     (property "Value" "10K" (id 1) (at 175.895 160.0539 90))
-    (property "Footprint" "" (id 2) (at 175.895 161.925 0)
+    (property "Footprint" "Resistor_SMD:R_0402_1005Metric" (id 2) (at 175.895 161.925 0)
       (effects (font (size 1.27 1.27)) hide)
     )
@@
       (effects (font (size 1.27 1.27)) (justify left))
     )
-    (property "Footprint" "" (id 2) (at 208.28 74.93 0)
+    (property "Footprint" "Resistor_SMD:R_0402_1005Metric" (id 2) (at 208.28 74.93 0)
       (effects (font (size 1.27 1.27)) hide)
     )
@@
       (effects (font (size 1.27 1.27)) (justify left))
     )
-    (property "Footprint" "" (id 2) (at 215.9 74.93 0)
+    (property "Footprint" "Resistor_SMD:R_0402_1005Metric" (id 2) (at 215.9 74.93 0)
       (effects (font (size 1.27 1.27)) hide)
     )
@@
     (property "Reference" "F2" (id 0) (at 203.2 63.1148 90))
     (property "Value" "Fuse" (id 1) (at 203.2 65.4135 90))
-    (property "Footprint" "" (id 2) (at 203.2 69.088 90)
+    (property "Footprint" "Fuse:Fuse_0603_1608Metric_Pad1.05x0.95mm_HandSolder" (id 2) (at 203.2 69.088 90)
       (effects (font (size 1.27 1.27)) hide)
     )
@@
       (effects (font (size 1.27 1.27)) (justify left))
     )
-    (property "Footprint" "" (id 2) (at 172.72 217.17 0)
+    (property "Footprint" "Capacitor_SMD:C_0402_1005Metric" (id 2) (at 172.72 217.17 0)
       (effects (font (size 1.27 1.27)) hide)
     )
@@
       (effects (font (size 1.27 1.27)) (justify left))
     )
-    (property "Footprint" "" (id 2) (at 181.61 217.17 0)
+    (property "Footprint" "Capacitor_SMD:C_0201_0603Metric" (id 2) (at 181.61 217.17 0)
       (effects (font (size 1.27 1.27)) hide)
     )
@@
       (effects (font (size 1.27 1.27)) (justify left))
     )
-    (property "Footprint" "" (id 2) (at 189.23 217.17 0)
+    (property "Footprint" "Capacitor_SMD:C_0402_1005Metric" (id 2) (at 189.23 217.17 0)
       (effects (font (size 1.27 1.27)) hide)
     )
@@
       (effects (font (size 1.27 1.27)) (justify left))
     )
-    (property "Footprint" "" (id 2) (at 196.85 217.17 0)
+    (property "Footprint" "Capacitor_SMD:C_0201_0603Metric" (id 2) (at 196.85 217.17 0)
       (effects (font (size 1.27 1.27)) hide)
     )
@@
       (effects (font (size 1.27 1.27)) (justify left))
     )
-    (property "Footprint" "" (id 2) (at 203.2 217.17 0)
+    (property "Footprint" "Capacitor_SMD:C_0402_1005Metric" (id 2) (at 203.2 217.17 0)
       (effects (font (size 1.27 1.27)) hide)
     )
@@
       (effects (font (size 1.27 1.27)) (justify left))
     )
-    (property "Footprint" "" (id 2) (at 209.55 217.17 0)
+    (property "Footprint" "Capacitor_SMD:C_0201_0603Metric" (id 2) (at 209.55 217.17 0)
       (effects (font (size 1.27 1.27)) hide)
     )
@@
       (effects (font (size 1.27 1.27)) (justify left))
     )
-    (property "Footprint" "" (id 2) (at 215.9 217.17 0)
+    (property "Footprint" "Capacitor_SMD:C_0201_0603Metric" (id 2) (at 215.9 217.17 0)
       (effects (font (size 1.27 1.27)) hide)
     )
@@
       (effects (font (size 1.27 1.27)) (justify left))
     )
-    (property "Footprint" "" (id 2) (at 222.25 217.17 0)
+    (property "Footprint" "Capacitor_SMD:C_0402_1005Metric" (id 2) (at 222.25 217.17 0)
       (effects (font (size 1.27 1.27)) hide)
     )
@@
       (effects (font (size 1.27 1.27)) (justify right))
     )
-    (property "Footprint" "" (id 2) (at 229.87 165.1 0)
+    (property "Footprint" "Diode_SMD:D_0402_1005Metric_Pad0.77x0.64mm_HandSolder" (id 2) (at 229.87 165.1 0)
       (effects (font (size 1.27 1.27)) hide)
     )
@@
     (property "Reference" "FB6" (id 0) (at 246.38 195.8552 90))
     (property "Value" "FerriteBead" (id 1) (at 246.38 198.1539 90))
-    (property "Footprint" "" (id 2) (at 246.38 203.708 90)
+    (property "Footprint" "Inductor_SMD:L_0402_1005Metric_Pad0.77x0.64mm_HandSolder" (id 2) (at 246.38 203.708 90)
       (effects (font (size 1.27 1.27)) hide)
     )
@@
     (property "Reference" "D35" (id 0) (at 189.23 83.0538 0))
     (property "Value" "PMEG3010CEJ" (id 1) (at 189.23 85.3525 0))
-    (property "Footprint" "" (id 2) (at 189.23 88.9 0)
+    (property "Footprint" "Diode_SMD:D_SOD-323F" (id 2) (at 189.23 88.9 0)
       (effects (font (size 1.27 1.27)) hide)
     )
@@
     (property "Reference" "D62" (id 0) (at 243.84 147.6968 0))
     (property "Value" "Protection-Diode" (id 1) (at 243.84 149.9955 0))
-    (property "Footprint" "" (id 2) (at 243.84 159.385 0)
+    (property "Footprint" "Package_SON:USON-10_2.5x1.0mm_P0.5mm" (id 2) (at 243.84 159.385 0)
       (effects (font (size 1.27 1.27)) hide)
     )
@@
     (pin "9")
   )
-  (symbol (lib_name "BeagleV:Protection-Diode_2") (lib_id "BeagleV:Protection-Diode") (at 262.89 159.385 0) (unit 2)
+  (symbol (lib_id "BeagleV:Protection-Diode") (at 262.89 159.385 0) (unit 2)
     (in_bom yes) (on_board yes) (fields_autoplaced)
     (property "Reference" "D62" (id 0) (at 262.89 147.6968 0))
     (property "Value" "Protection-Diode" (id 1) (at 262.89 149.9955 0))
-    (property "Footprint" "" (id 2) (at 262.89 159.385 0)
+    (property "Footprint" "Package_SON:USON-10_2.5x1.0mm_P0.5mm" (id 2) (at 262.89 159.385 0)
       (effects (font (size 1.27 1.27)) hide)
     )
@@
     (pin "8")
   )
-  (symbol (lib_name "BeagleV:Protection-Diode_1") (lib_id "BeagleV:Protection-Diode") (at 282.575 159.385 0) (unit 1)
+  (symbol (lib_id "BeagleV:Protection-Diode") (at 282.575 159.385 0) (unit 1)
     (in_bom yes) (on_board yes) (fields_autoplaced)
     (property "Reference" "D63" (id 0) (at 282.575 147.6968 0))
     (property "Value" "Protection-Diode" (id 1) (at 282.575 149.9955 0))
-    (property "Footprint" "" (id 2) (at 282.575 159.385 0)
+    (property "Footprint" "Package_SON:USON-10_2.5x1.0mm_P0.5mm" (id 2) (at 282.575 159.385 0)
       (effects (font (size 1.27 1.27)) hide)
     )
@@
     (pin "9")
   )
-  (symbol (lib_name "BeagleV:Protection-Diode_2") (lib_id "BeagleV:Protection-Diode") (at 301.625 159.385 0) (unit 2)
+  (symbol (lib_id "BeagleV:Protection-Diode") (at 301.625 159.385 0) (unit 2)
     (in_bom yes) (on_board yes) (fields_autoplaced)
     (property "Reference" "D63" (id 0) (at 301.625 147.6968 0))
     (property "Value" "Protection-Diode" (id 1) (at 301.625 149.9955 0))
-    (property "Footprint" "" (id 2) (at 301.625 159.385 0)
+    (property "Footprint" "Package_SON:USON-10_2.5x1.0mm_P0.5mm" (id 2) (at 301.625 159.385 0)
       (effects (font (size 1.27 1.27)) hide)
     )
@@
     (pin "8")
   )
-  (symbol (lib_name "BeagleV:Protection-Diode_1") (lib_id "BeagleV:Protection-Diode") (at 323.215 159.385 0) (unit 1)
+  (symbol (lib_id "BeagleV:Protection-Diode") (at 323.215 159.385 0) (unit 1)
     (in_bom yes) (on_board yes) (fields_autoplaced)
     (property "Reference" "D64" (id 0) (at 323.215 147.6968 0))
     (property "Value" "Protection-Diode" (id 1) (at 323.215 149.9955 0))
-    (property "Footprint" "" (id 2) (at 323.215 159.385 0)
+    (property "Footprint" "Package_SON:USON-10_2.5x1.0mm_P0.5mm" (id 2) (at 323.215 159.385 0)
       (effects (font (size 1.27 1.27)) hide)
     )
@@
     (pin "9")
   )
-  (symbol (lib_name "BeagleV:Protection-Diode_2") (lib_id "BeagleV:Protection-Diode") (at 342.265 159.385 0) (unit 2)
+  (symbol (lib_id "BeagleV:Protection-Diode") (at 342.265 159.385 0) (unit 2)
     (in_bom yes) (on_board yes) (fields_autoplaced)
     (property "Reference" "D64" (id 0) (at 342.265 147.6968 0))
     (property "Value" "Protection-Diode" (id 1) (at 342.265 149.9955 0))
-    (property "Footprint" "" (id 2) (at 342.265 159.385 0)
+    (property "Footprint" "Package_SON:USON-10_2.5x1.0mm_P0.5mm" (id 2) (at 342.265 159.385 0)
       (effects (font (size 1.27 1.27)) hide)
     )
@@
       (effects (font (size 1.27 1.27)) (justify left))
     )
-    (property "Footprint" "" (id 2) (at 379.73 119.38 0)
+    (property "Footprint" "BeagleV:HDMI-Type-A" (id 2) (at 379.73 119.38 0)
       (effects (font (size 1.27 1.27)) hide)
     )
@@
     (property "Reference" "U11" (id 0) (at 131.445 86.7876 0))
     (property "Value" "TDA19988" (id 1) (at 131.445 89.0863 0))
-    (property "Footprint" "" (id 2) (at 135.89 160.02 0)
-      (effects (font (size 1.27 1.27)) hide)
-    )
+    (property "Footprint" "BeagleV:TDA19988-QFN-64_EP_9x9_Pitch0.5mm" (id 2) (at 135.89 160.02 0)
+      (effects (font (size 1.27 1.27)) hide)
+    )
