File: BeagleV/BeagleV_LPDDR_A.kicad_sch (KiCad schematic)
At the start: 80 parts, among them U7 32Gbit_RAM

Commit message: Initial commit to working branch, Cloned from the gitlab repository
Parts:
- C48, C68: footprint (none) -> Capacitor_SMD:C_0603_1608Metric
- C49, C59, C60, C67, C69, C79: footprint (none) -> Capacitor_SMD:C_0402_1005Metric
- C50, C51, C52, C53, C54, C55, C56, C57, C58, C61, C62, C63, C64, C65, C66, C70, C71, C72, C73, C74, C75, C76, C77, C78: footprint (none) -> Capacitor_SMD:C_0201_0603Metric
- R184, R62, R64, R65, R66, R67, R68, R69, R70: footprint (none) -> Resistor_SMD:R_0402_1005Metric
- U7: footprint (none) -> BeagleV:LPDDR4-200-WFBGA-10x14.5
- gave numbers to parts that had none: 14
