File: BeagleV/BeagleV_LPDDR_B.kicad_sch (KiCad schematic)
At the start: 80 parts, among them U8 32Gbit_RAM

Commit message: Initial commit to working branch, Cloned from the gitlab repository
Parts:
- C100, C80: footprint (none) -> Capacitor_SMD:C_0603_1608Metric
- C101, C111, C81, C91, C92, C99: footprint (none) -> Capacitor_SMD:C_0402_1005Metric
- C102, C103, C104, C105, C106, C107, C108, C109, C110, C82, C83, C84, C85, C86, C87, C88, C89, C90, C93, C94, C95, C96, C97, C98: footprint (none) -> Capacitor_SMD:C_0201_0603Metric
- R71, R72, R73, R74, R75, R76, R78, R79: footprint (none) -> Resistor_SMD:R_0402_1005Metric
- R77: value DNP -> 10K; footprint (none) -> Resistor_SMD:R_0402_1005Metric
- U8: footprint (none) -> BeagleV:LPDDR4-200-WFBGA-10x14.5
- gave numbers to parts that had none: 14
