File: BeagleV/BeagleV_PMIC.kicad_sch (KiCad schematic)
At the start: 78 parts, among them Q6 CSD87381P, Q7 CSD87381P, SW2 Tactile-Switch, U13 LMR62014, U14 TPS65086100

Commit message: Initial commit to working branch, Cloned from the gitlab repository
Parts:
- removed P? (x2): VCC_0V9, symbol BeagleV:VCC_0V9
- removed P? (x2): LDO_3V3, symbol BeagleV:LDO_3V3
- removed P? (x3): VSYS_5V8, symbol BeagleV:VSYS_5V8
- removed P?: VDD2PEN_OTP_1V8, symbol BeagleV:VDD2PEN_OTP_1V8
- C222, C250, C288, C296, C298, C302, C306, C307: footprint (none) -> Capacitor_SMD:C_0402_1005Metric
- C248, C249, C27, C273, C274, C275, C276, C283, C284, C289, C290, C291, C293, C294, C295, C301, C303, C304, C308: footprint (none) -> Capacitor_SMD:C_0603_1608Metric
- C277, C282, C286, C287, C297, C300, C305: footprint (none) -> Capacitor_SMD:C_0201_0603Metric
- D5: footprint (none) -> Diode_SMD:D_0402_1005Metric_Pad0.77x0.64mm_HandSolder
- L1, L7, L8: footprint (none) -> BeagleV:WPN201610H_2x1.6
- L4, L5: footprint (none) -> BeagleV:Codaca_4.4x4.4
- L6: footprint (none) -> Inductor_SMD:L_0805_2012Metric_Pad1.05x1.20mm_HandSolder
- Q6, Q7: footprint (none) -> BeagleV:CSD87381P
- R117, R118, R119, R121, R142, R166, R252, R254, R255, R256, R257, R258, R259, R260, R261, R262, R263, R264, R63: footprint (none) -> Resistor_SMD:R_0402_1005Metric
- SW2: footprint (none) -> BeagleV:switch
- U13: footprint (none) -> BeagleV:DBV0005A-SOT-23
- U14: footprint (none) -> BeagleV:TPS650861-QFN-64_EP_8.15x8.15_Pitch0.4mm
Connections:
- net +1V1: no longer C222.1, C222.2, C248.1, C249.1, C249.2, C250.1, C27.1, C273.1, C274.1, C275.1, C275.2, C276.1, C276.2, C282.1, C283.1, C283.2, C284.1, C284.2, C286.1, C286.2, C287.1, C287.2, C288.1, C288.2, C289.1, C289.2, C290.1, C290.2, C291.1, C291.2, C293.1, C293.2, C294.1, C294.2, C295.1, C295.2, C296.1, C297.1, C298.1, C300.1, C300.2, C301.1, C301.2, C302.1, C303.1, C303.2, C304.1, C304.2, C305.1, C306.1, C307.1, C308.1, C308.2, D5.1 (A1), D65.1 (K), L4.2, L6.1, L8.2, Q6.2, Q6.3, Q7.2, Q7.3, R117.1, R118.1, R142.1, R252.1, R256.2, R258.1, R258.2, R261.1, R262.2, R263.1, R264.2, SW2.1, SW2.3, U13.2 (GND), U13.5 (VIN), U14.1 (FBGND2), U14.11 (PVIN3), U14.14 (CTL6_SLPENB2), U14.18 (PVINSWB1_B2), U14.21 (PVIN5), U14.23 (FB4), U14.24 (PVIN4), U14.29 (FBVOUT1), U14.30 (ILIM1), U14.31 (SWA1), U14.34 (SW1), U14.36 (PGNDSNS1), U14.38 (DRV5V_1_6), U14.40 (PGNDSNS6), U14.44 (FBVOUT6), U14.46 (PVIBVTT), U14.48 (VTTFB), U14.50 (PVINLDOA2_A3), U14.52 (AGND), U14.55 (VSYS), U14.57 (V5ANA), U14.6 (PGNDSNS2), U14.61 (CTL3_SLPENB1), U14.65 (PAD), U14.8 (DRV5V_2_A1), U14.9 (LDOA1)
- net +1V8: now reaches C296.2, U14.32 (PVINSWA1)
- net +1V8: now also C275.2, C276.2, L8.2, U14.23 (FB4)
- new net +5V: C249.2, C283.2, C284.2, C289.2, C290.2, C291.2, C293.2, C294.2, C295.2, C303.1, C308.2, L6.1, Q6.2, Q7.2, R263.1, U13.5 (VIN), U14.11 (PVIN3), U14.21 (PVIN5), U14.24 (PVIN4), U14.38 (DRV5V_1_6), U14.57 (V5ANA), U14.8 (DRV5V_2_A1)
- new net GND: C222.1, C248.1, C249.1, C250.1, C27.1, C273.1, C274.1, C275.1, C276.1, C282.1, C283.1, C284.1, C286.1, C287.1, C288.1, C289.1, C290.1, C291.1, C293.1, C294.1, C295.1, C296.1, C297.1, C298.1, C300.1, C301.1, C303.2, C304.2, C305.1, C306.1, C307.1, C308.1, D5.1 (A1), Q6.3, Q7.3, R142.1, R256.2, R258.2, R262.2, R264.2, SW2.1, SW2.3, U13.2 (GND), U14.1 (FBGND2), U14.14 (CTL6_SLPENB2), U14.18 (PVINSWB1_B2), U14.29 (FBVOUT1), U14.30 (ILIM1), U14.34 (SW1), U14.36 (PGNDSNS1), U14.40 (PGNDSNS6), U14.48 (VTTFB), U14.50 (PVINLDOA2_A3), U14.52 (AGND), U14.6 (PGNDSNS2), U14.61 (CTL3_SLPENB1), U14.65 (PAD)
- new net LDO_3V3: C222.2, R117.1, R118.1, R252.1, U14.9 (LDOA1)
- new net VCC_0V9: C286.2, C287.2, C288.2, L4.2, U14.44 (FBVOUT6), U14.46 (PVIBVTT)
- new net VDD2PEN_OTP_1V8: C300.2, R258.1, U14.31 (SWA1)
- new net VSYS_5V8: C301.2, C302.1, C304.1, D65.1 (K), R261.1, U14.55 (VSYS)
