File: BeagleV/BeagleV_RPI_Conn.kicad_sch (KiCad schematic)
At the start: 19 parts, among them J12 JTAG-Connector, J14 DNP Conn_01x03_Male, J7 PI-Connector-2x20-2.54mm, Q1 CJ1012, Q3 CJ1012, SW3 Tactile-Switch

Commit message: Initial commit to working branch, Cloned from the gitlab repository
Parts:
- removed P? (x2): USB_5V, symbol BeagleV:USB_5V
- D6: footprint (none) -> Diode_SMD:D_SOD-323F
- J12: footprint (none) -> Connector:Tag-Connect_TC2050-IDC-NL_2x05_P1.27mm_Vertical
- J14: footprint (none) -> Connector_PinHeader_2.54mm:PinHeader_1x03_P2.54mm_Vertical
- J7: footprint (none) -> Connector_PinHeader_2.54mm:PinHeader_2x20_P2.54mm_Vertical
- LED1, LED2: footprint (none) -> LED_SMD:LED_0603_1608Metric_Pad1.05x0.95mm_HandSolder
- Q1, Q3: footprint (none) -> Package_TO_SOT_SMD:SOT-523
- R100: value 100K -> 10K; footprint (none) -> Resistor_SMD:R_0402_1005Metric
- R159, R160, R161, R167, R2, R3, R4: footprint (none) -> Resistor_SMD:R_0402_1005Metric
- SW3: footprint (none) -> BeagleV:switch
Connections:
- net LDO_3V3: no longer names the net of R2.2
- net LDO_3V3: no longer R3.2
