File: BeagleV/BeagleV_Type_C_uSD.kicad_sch (KiCad schematic)
At the start: 38 parts, among them J10 MICRO_SD_ST_TF_003A_16_1x14_5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, J13 USB_TYPE_C, Q8 IRLML6401, Q9 BCM857BS-7F-F, U16 256MBit_NOR_FLASH

Commit message: Initial commit to working branch, Cloned from the gitlab repository
Parts:
- removed P?: USB_5V, symbol BeagleV:USB_5V
- C198, C278, C280: footprint (none) -> Capacitor_SMD:C_0402_1005Metric
- C199, C279, C281: footprint (none) -> Capacitor_SMD:C_0201_0603Metric
- D52: footprint (none) -> Diode_SMD:D_SMB
- J10: footprint (none) -> BeagleV:ST-TF-003A
- J13: footprint (none) -> BeagleV:USB-Type-C
- Q9: footprint (none) -> Package_TO_SOT_SMD:SOT-363_SC-70-6_Handsoldering
- R1, R102, R103, R104, R105, R106, R107, R123, R124, R125, R126, R134, R147, R232, R233, R234, R235, R236, R237, R238: footprint (none) -> Resistor_SMD:R_0201_0603Metric
- R101, R162, R163, R248, R249: footprint (none) -> Resistor_SMD:R_0402_1005Metric
- U16: value 256MBit_NOR_FLASH -> GD25LQ256DWIGR; footprint (none) -> BeagleV:GD25LQ256D
Connections:
- net LDO_3V3: no longer names the net of D52.2 (A2), J13.B4 (A9/B4/VBUS), J13.B9 (A4/B9/VBUS), Q8.3 (D), Q9.1
Other:
- note added: "256MBit_NOR_FLASH"
