File: BeagleV/BeagleV_USB_3_HUB.kicad_sch (KiCad schematic)
At the start: 45 parts, among them U1 GL3520-OS322, X1 25MHz

Commit message: Initial commit to working branch, Cloned from the gitlab repository
Parts:
- C10, C22, C23, C246, C247, C4: footprint (none) -> Capacitor_SMD:C_0402_1005Metric
- C11, C12, C13, C14, C15, C16, C17, C18, C185, C186, C237, C238, C239, C24, C240, C241, C242, C243, C244, C245, C5, C6, C7, C8, C9: footprint (none) -> Capacitor_SMD:C_0201_0603Metric
- FB4: footprint (none) -> Inductor_SMD:L_0402_1005Metric_Pad0.77x0.64mm_HandSolder
- R143, R144, R146, R165, R23, R25, R26: footprint (none) -> Resistor_SMD:R_0402_1005Metric
- U1: footprint (none) -> BeagleV:GL3520-22-QFN-64_EP_8x8_Pitch0.4mm
- X1: footprint (none) -> BeagleV:SMCE-2520
Connections:
- net GND: now also X1.2, X1.4; no longer X1.1, X1.3
- net at C246.2, R143.1, U1.3 (X1): now also X1.1; no longer X1.2
- net at C247.2, R143.2, U1.4 (X2): now also X1.3; no longer X1.4
