File: BeagleV/BeagleV_USB_Type_A_A.kicad_sch (KiCad schematic)
At the start: 12 parts, among them J4 USB-TYPE-A-3.0, Q2 CJ1012, U2 ETA6020D2G

Commit message: Initial commit to working branch, Cloned from the gitlab repository
Parts:
- removed P?: VCC_5V_USB, symbol BeagleV:VCC_5V_USB
- C19, C20: footprint (none) -> Capacitor_SMD:C_0201_0603Metric
- C21: footprint (none) -> Capacitor_SMD:C_1206_3216Metric
- D27, D28, D29: footprint (none) -> BeagleV:PCMF2USB3S
- J4: footprint (none) -> BeagleV:Stacked-USB-TypeA
- Q2: footprint (none) -> Package_TO_SOT_SMD:SOT-523
- R138, R24: footprint (none) -> Resistor_SMD:R_0402_1005Metric
- U2: footprint (none) -> BeagleV:ETA6020-DFN2x2-6L
Connections:
- net LDO_3V3 renamed VCC_5V_USB
Changed lines of the file:
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@@
   (title_block
     (title "Beagle V")
-    (date "2021-06-03")
+    (date "2021-06-11")
     (rev "v0.7")
   )
@@
   (symbol (lib_id "BeagleV:VCC_5V_USB") (at 290.83 48.26 0) (unit 1)
     (in_bom yes) (on_board yes)
-    (property "Reference" "P?" (id 0) (at 290.83 48.26 0)
+    (property "Reference" "#P023" (id 0) (at 290.83 48.26 0)
       (effects (font (size 1.27 1.27)) hide)
     )
@@
     (property "Reference" "R138" (id 0) (at 208.28 54.2502 90))
     (property "Value" "10K" (id 1) (at 208.28 56.5489 90))
-    (property "Footprint" "" (id 2) (at 208.28 58.42 0)
+    (property "Footprint" "Resistor_SMD:R_0402_1005Metric" (id 2) (at 208.28 58.42 0)
       (effects (font (size 1.27 1.27)) hide)
     )
@@
       (effects (font (size 1.27 1.27)) (justify right))
     )
-    (property "Footprint" "" (id 2) (at 236.22 67.31 0)
+    (property "Footprint" "Resistor_SMD:R_0402_1005Metric" (id 2) (at 236.22 67.31 0)
       (effects (font (size 1.27 1.27)) hide)
     )
@@
       (effects (font (size 1.27 1.27)) (justify left))
     )
-    (property "Footprint" "" (id 2) (at 220.98 67.31 0)
+    (property "Footprint" "Capacitor_SMD:C_0201_0603Metric" (id 2) (at 220.98 67.31 0)
       (effects (font (size 1.27 1.27)) hide)
     )
@@
       (effects (font (size 1.27 1.27)) (justify left))
     )
-    (property "Footprint" "" (id 2) (at 273.05 62.23 0)
+    (property "Footprint" "Capacitor_SMD:C_0201_0603Metric" (id 2) (at 273.05 62.23 0)
       (effects (font (size 1.27 1.27)) hide)
     )
@@
       (effects (font (size 1.27 1.27)) (justify left))
     )
-    (property "Footprint" "" (id 2) (at 279.4 62.23 0)
+    (property "Footprint" "Capacitor_SMD:C_1206_3216Metric" (id 2) (at 279.4 62.23 0)
       (effects (font (size 1.27 1.27)) hide)
     )
@@
       (effects (font (size 1.27 1.27)) (justify left))
     )
-    (property "Footprint" "" (id 2) (at 106.41 75.39 0)
+    (property "Footprint" "Package_TO_SOT_SMD:SOT-523" (id 2) (at 106.41 75.39 0)
       (effects (font (size 1.27 1.27)) hide)
     )
@@
     (property "Reference" "D27" (id 0) (at 119.38 95.7776 0))
     (property "Value" "PCMF2USB3S" (id 1) (at 125.73 98.0763 0))
-    (property "Footprint" "" (id 2) (at 149.86 114.3 0)
+    (property "Footprint" "BeagleV:PCMF2USB3S" (id 2) (at 149.86 114.3 0)
       (effects (font (size 1.27 1.27)) hide)
     )
@@
     (property "Reference" "D28" (id 0) (at 119.38 116.0976 0))
     (property "Value" "PCMF2USB3S" (id 1) (at 125.73 118.3963 0))
-    (property "Footprint" "" (id 2) (at 149.86 134.62 0)
+    (property "Footprint" "BeagleV:PCMF2USB3S" (id 2) (at 149.86 134.62 0)
       (effects (font (size 1.27 1.27)) hide)
     )
@@
     (property "Reference" "D27" (id 0) (at 119.38 156.7376 0))
     (property "Value" "PCMF2USB3S" (id 1) (at 125.73 159.0363 0))
-    (property "Footprint" "" (id 2) (at 149.86 175.26 0)
+    (property "Footprint" "BeagleV:PCMF2USB3S" (id 2) (at 149.86 175.26 0)
       (effects (font (size 1.27 1.27)) hide)
     )
@@
     (property "Reference" "D28" (id 0) (at 119.38 177.0576 0))
     (property "Value" "PCMF2USB3S" (id 1) (at 125.73 179.3563 0))
-    (property "Footprint" "" (id 2) (at 149.86 195.58 0)
+    (property "Footprint" "BeagleV:PCMF2USB3S" (id 2) (at 149.86 195.58 0)
       (effects (font (size 1.27 1.27)) hide)
     )
@@
     (property "Reference" "D29" (id 0) (at 118.11 198.6476 0))
     (property "Value" "PCMF2USB3S" (id 1) (at 125.73 200.9463 0))
-    (property "Footprint" "" (id 2) (at 149.86 217.17 0)
+    (property "Footprint" "BeagleV:PCMF2USB3S" (id 2) (at 149.86 217.17 0)
       (effects (font (size 1.27 1.27)) hide)
     )
@@
     (property "Reference" "D29" (id 0) (at 119.38 136.4176 0))
     (property "Value" "PCMF2USB3S" (id 1) (at 127 138.7163 0))
-    (property "Footprint" "" (id 2) (at 151.13 154.94 0)
+    (property "Footprint" "BeagleV:PCMF2USB3S" (id 2) (at 151.13 154.94 0)
       (effects (font (size 1.27 1.27)) hide)
     )
@@
     (property "Reference" "U2" (id 0) (at 251.46 50.7196 0))
     (property "Value" "ETA6020D2G" (id 1) (at 251.46 53.0183 0))
-    (property "Footprint" "" (id 2) (at 248.92 60.96 0)
+    (property "Footprint" "BeagleV:ETA6020-DFN2x2-6L" (id 2) (at 248.92 60.96 0)
       (effects (font (size 1.27 1.27)) hide)
     )
@@
       (effects (font (size 1.27 1.27)) (justify left))
     )
-    (property "Footprint" "" (id 2) (at 317.5 152.4 0)
-      (effects (font (size 1.27 1.27)) hide)
-    )
+    (property "Footprint" "BeagleV:Stacked-USB-TypeA" (id 2) (at 317.5 152.4 0)
+      (effects (font (size 1.27 1.27)) hide)
+    )
