File: BeagleV/BeagleV_USB_Type_A_B.kicad_sch (KiCad schematic)
At the start: 7 parts, among them J5 USB-TYPE-A-3.0

Commit message: Initial commit to working branch, Cloned from the gitlab repository
Parts:
- removed P?: VCC_5V_USB, symbol BeagleV:VCC_5V_USB
- C25: footprint (none) -> Capacitor_SMD:C_0201_0603Metric
- C26: footprint (none) -> Capacitor_SMD:C_1206_3216Metric
- D30, D31, D32: footprint (none) -> BeagleV:PCMF2USB3S
- J5: footprint (none) -> BeagleV:Stacked-USB-TypeA
Connections:
- net LDO_3V3 renamed VCC_5V_USB
Changed lines of the file:
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@@
   (title_block
     (title "Beagle V")
-    (date "2021-06-03")
+    (date "2021-06-11")
     (rev "v0.7")
   )
@@
   (symbol (lib_id "BeagleV:VCC_5V_USB") (at 289.56 92.71 0) (unit 1)
     (in_bom yes) (on_board yes)
-    (property "Reference" "P?" (id 0) (at 289.56 92.71 0)
+    (property "Reference" "#P024" (id 0) (at 289.56 92.71 0)
       (effects (font (size 1.27 1.27)) hide)
     )
@@
       (effects (font (size 1.27 1.27)) (justify left))
     )
-    (property "Footprint" "" (id 2) (at 289.56 103.505 0)
+    (property "Footprint" "Capacitor_SMD:C_0201_0603Metric" (id 2) (at 289.56 103.505 0)
       (effects (font (size 1.27 1.27)) hide)
     )
@@
       (effects (font (size 1.27 1.27)) (justify left))
     )
-    (property "Footprint" "" (id 2) (at 295.275 103.505 0)
+    (property "Footprint" "Capacitor_SMD:C_1206_3216Metric" (id 2) (at 295.275 103.505 0)
       (effects (font (size 1.27 1.27)) hide)
     )
@@
     (property "Reference" "D30" (id 0) (at 129.54 107.2076 0))
     (property "Value" "PCMF2USB3S" (id 1) (at 135.89 109.5063 0))
-    (property "Footprint" "" (id 2) (at 160.02 125.73 0)
+    (property "Footprint" "BeagleV:PCMF2USB3S" (id 2) (at 160.02 125.73 0)
       (effects (font (size 1.27 1.27)) hide)
     )
@@
     (property "Reference" "D31" (id 0) (at 129.54 127.5276 0))
     (property "Value" "PCMF2USB3S" (id 1) (at 135.89 129.8263 0))
-    (property "Footprint" "" (id 2) (at 160.02 146.05 0)
+    (property "Footprint" "BeagleV:PCMF2USB3S" (id 2) (at 160.02 146.05 0)
       (effects (font (size 1.27 1.27)) hide)
     )
@@
     (property "Reference" "D32" (id 0) (at 130.81 147.8476 0))
     (property "Value" "PCMF2USB3S" (id 1) (at 135.89 150.1463 0))
-    (property "Footprint" "" (id 2) (at 160.02 166.37 0)
+    (property "Footprint" "BeagleV:PCMF2USB3S" (id 2) (at 160.02 166.37 0)
       (effects (font (size 1.27 1.27)) hide)
     )
@@
     (property "Reference" "D30" (id 0) (at 129.54 168.1676 0))
     (property "Value" "PCMF2USB3S" (id 1) (at 135.89 170.4663 0))
-    (property "Footprint" "" (id 2) (at 160.02 186.69 0)
+    (property "Footprint" "BeagleV:PCMF2USB3S" (id 2) (at 160.02 186.69 0)
       (effects (font (size 1.27 1.27)) hide)
     )
@@
     (property "Reference" "D31" (id 0) (at 129.54 188.4876 0))
     (property "Value" "PCMF2USB3S" (id 1) (at 135.89 190.7863 0))
-    (property "Footprint" "" (id 2) (at 160.02 207.01 0)
+    (property "Footprint" "BeagleV:PCMF2USB3S" (id 2) (at 160.02 207.01 0)
       (effects (font (size 1.27 1.27)) hide)
     )
@@
     (property "Reference" "D32" (id 0) (at 130.81 210.0776 0))
     (property "Value" "PCMF2USB3S" (id 1) (at 135.89 212.3763 0))
-    (property "Footprint" "" (id 2) (at 160.02 228.6 0)
+    (property "Footprint" "BeagleV:PCMF2USB3S" (id 2) (at 160.02 228.6 0)
       (effects (font (size 1.27 1.27)) hide)
     )
@@
     (property "Reference" "J5" (id 0) (at 311.785 110.9176 0))
     (property "Value" "USB-TYPE-A-3.0" (id 1) (at 319.405 212.2763 0))
-    (property "Footprint" "" (id 2) (at 327.66 163.83 0)
-      (effects (font (size 1.27 1.27)) hide)
-    )
+    (property "Footprint" "BeagleV:Stacked-USB-TypeA" (id 2) (at 327.66 163.83 0)
+      (effects (font (size 1.27 1.27)) hide)
+    )
