File: BeagleV/BeagleV_VIC_ChipLink.kicad_sch (KiCad schematic)
At the start: 18 parts, among them U9 VIC-V10

Commit message: Initial commit to working branch, Cloned from the gitlab repository
Parts:
- C177, C178, C182: footprint (none) -> Capacitor_SMD:C_0402_1005Metric
- C179, C180, C181, C183, C184: footprint (none) -> Capacitor_SMD:C_0201_0603Metric
- R110, R113, R156, R157, R158: footprint (none) -> Resistor_SMD:R_0201_0603Metric
- R127, R128, R129, R131: footprint (none) -> Resistor_SMD:R_0402_1005Metric
- U9: footprint (none) -> BeagleV:JH7100 - BGA-961_31x31_20.5x20.5mm
Other:
- moved on the sheet: U9I, U9J
Changed lines of the file:
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@@
   (title_block
     (title "Beagle V")
-    (date "2021-06-03")
+    (date "2021-06-11")
     (rev "v0.7")
   )
@@
     (property "Reference" "R110" (id 0) (at 126.365 145.6902 90))
     (property "Value" "33R" (id 1) (at 135.255 146.7189 90))
-    (property "Footprint" "" (id 2) (at 131.445 147.32 0)
+    (property "Footprint" "Resistor_SMD:R_0201_0603Metric" (id 2) (at 131.445 147.32 0)
       (effects (font (size 1.27 1.27)) hide)
     )
@@
     (property "Reference" "R113" (id 0) (at 126.365 148.2302 90))
     (property "Value" "33R" (id 1) (at 135.255 149.2589 90))
-    (property "Footprint" "" (id 2) (at 131.445 149.86 0)
+    (property "Footprint" "Resistor_SMD:R_0201_0603Metric" (id 2) (at 131.445 149.86 0)
       (effects (font (size 1.27 1.27)) hide)
     )
@@
     (property "Reference" "R156" (id 0) (at 126.365 150.7702 90))
     (property "Value" "33R" (id 1) (at 135.255 151.7989 90))
-    (property "Footprint" "" (id 2) (at 131.445 152.4 0)
+    (property "Footprint" "Resistor_SMD:R_0201_0603Metric" (id 2) (at 131.445 152.4 0)
       (effects (font (size 1.27 1.27)) hide)
     )
@@
     (property "Reference" "R157" (id 0) (at 126.365 153.3102 90))
     (property "Value" "33R" (id 1) (at 135.255 154.3389 90))
-    (property "Footprint" "" (id 2) (at 131.445 154.94 0)
+    (property "Footprint" "Resistor_SMD:R_0201_0603Metric" (id 2) (at 131.445 154.94 0)
       (effects (font (size 1.27 1.27)) hide)
     )
@@
     (property "Reference" "R158" (id 0) (at 126.365 163.4702 90))
     (property "Value" "33R" (id 1) (at 135.255 164.4989 90))
-    (property "Footprint" "" (id 2) (at 131.445 165.1 0)
+    (property "Footprint" "Resistor_SMD:R_0201_0603Metric" (id 2) (at 131.445 165.1 0)
       (effects (font (size 1.27 1.27)) hide)
     )
@@
       (effects (font (size 1.27 1.27)) (justify left))
     )
-    (property "Footprint" "" (id 2) (at 242.57 59.69 0)
+    (property "Footprint" "Resistor_SMD:R_0402_1005Metric" (id 2) (at 242.57 59.69 0)
       (effects (font (size 1.27 1.27)) hide)
     )
@@
       (effects (font (size 1.27 1.27)) (justify left))
     )
-    (property "Footprint" "" (id 2) (at 247.65 59.69 0)
+    (property "Footprint" "Resistor_SMD:R_0402_1005Metric" (id 2) (at 247.65 59.69 0)
       (effects (font (size 1.27 1.27)) hide)
     )
@@
       (effects (font (size 1.27 1.27)) (justify left))
     )
-    (property "Footprint" "" (id 2) (at 252.73 59.69 0)
+    (property "Footprint" "Resistor_SMD:R_0402_1005Metric" (id 2) (at 252.73 59.69 0)
       (effects (font (size 1.27 1.27)) hide)
     )
@@
       (effects (font (size 1.27 1.27)) (justify left))
     )
-    (property "Footprint" "" (id 2) (at 257.81 59.69 0)
+    (property "Footprint" "Resistor_SMD:R_0402_1005Metric" (id 2) (at 257.81 59.69 0)
       (effects (font (size 1.27 1.27)) hide)
     )
@@
       (effects (font (size 1.27 1.27)) (justify left))
     )
-    (property "Footprint" "" (id 2) (at 72.39 209.55 0)
+    (property "Footprint" "Capacitor_SMD:C_0402_1005Metric" (id 2) (at 72.39 209.55 0)
       (effects (font (size 1.27 1.27)) hide)
     )
@@
       (effects (font (size 1.27 1.27)) (justify left))
     )
-    (property "Footprint" "" (id 2) (at 72.39 246.38 0)
+    (property "Footprint" "Capacitor_SMD:C_0402_1005Metric" (id 2) (at 72.39 246.38 0)
       (effects (font (size 1.27 1.27)) hide)
     )
@@
       (effects (font (size 1.27 1.27)) (justify left))
     )
-    (property "Footprint" "" (id 2) (at 78.74 209.55 0)
+    (property "Footprint" "Capacitor_SMD:C_0402_1005Metric" (id 2) (at 78.74 209.55 0)
       (effects (font (size 1.27 1.27)) hide)
     )
@@
       (effects (font (size 1.27 1.27)) (justify left))
     )
-    (property "Footprint" "" (id 2) (at 78.74 246.38 0)
+    (property "Footprint" "Capacitor_SMD:C_0201_0603Metric" (id 2) (at 78.74 246.38 0)
       (effects (font (size 1.27 1.27)) hide)
     )
@@
       (effects (font (size 1.27 1.27)) (justify left))
     )
-    (property "Footprint" "" (id 2) (at 85.09 209.55 0)
+    (property "Footprint" "Capacitor_SMD:C_0201_0603Metric" (id 2) (at 85.09 209.55 0)
       (effects (font (size 1.27 1.27)) hide)
     )
@@
       (effects (font (size 1.27 1.27)) (justify left))
     )
-    (property "Footprint" "" (id 2) (at 85.09 246.38 0)
+    (property "Footprint" "Capacitor_SMD:C_0201_0603Metric" (id 2) (at 85.09 246.38 0)
       (effects (font (size 1.27 1.27)) hide)
     )
@@
       (effects (font (size 1.27 1.27)) (justify left))
     )
-    (property "Footprint" "" (id 2) (at 91.44 209.55 0)
+    (property "Footprint" "Capacitor_SMD:C_0201_0603Metric" (id 2) (at 91.44 209.55 0)
       (effects (font (size 1.27 1.27)) hide)
     )
@@
       (effects (font (size 1.27 1.27)) (justify left))
     )
-    (property "Footprint" "" (id 2) (at 97.79 209.55 0)
+    (property "Footprint" "Capacitor_SMD:C_0201_0603Metric" (id 2) (at 97.79 209.55 0)
       (effects (font (size 1.27 1.27)) hide)
     )
@@
     (property "Reference" "U9" (id 0) (at 241.935 196.0076 0))
     (property "Value" "VIC-V10" (id 1) (at 241.935 198.3063 0))
-    (property "Footprint" "" (id 2) (at 226.98 164.91 0)
+    (property "Footprint" "BeagleV:JH7100 - BGA-961_31x31_20.5x20.5mm" (id 2) (at 226.98 164.91 0)
       (effects (font (size 1.27 1.27)) hide)
     )
@@
     (pin "AL5")
   )
-  (symbol (lib_name "BeagleV:VIC-V10_1") (lib_id "BeagleV:VIC-V10") (at 186.69 118.11 0) (unit 9)
+  (symbol (lib_id "BeagleV:VIC-V10") (at 186.69 118.11 0) (unit 9)
     (in_bom yes) (on_board yes) (fields_autoplaced)
     (property "Reference" "U9" (id 0) (at 186.69 45.2276 0))
     (property "Value" "VIC-V10" (id 1) (at 186.69 47.5263 0))
-    (property "Footprint" "" (id 2) (at 167.29 50.61 0)
-      (effects (font (size 1.27 1.27)) hide)
-    )
+    (property "Footprint" "BeagleV:JH7100 - BGA-961_31x31_20.5x20.5mm" (id 2) (at 167.29 50.61 0)
+      (effects (font (size 1.27 1.27)) hide)
+    )
