File: BeagleV/BeagleV_VIC_DDR_Ctrl.kicad_sch (KiCad schematic)
At the start: 13 parts, among them U9 VIC-V10

Commit message: Initial commit to working branch, Cloned from the gitlab repository
Parts:
- R80, R81, R82, R83: footprint (none) -> Resistor_SMD:R_0402_1005Metric
- U9: footprint (none) -> BeagleV:JH7100 - BGA-961_31x31_20.5x20.5mm
Other:
- moved on the sheet: U9E, U9F
Changed lines of the file:
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@@
   (title_block
     (title "Beagle V")
-    (date "2021-06-03")
+    (date "2021-06-11")
     (rev "v0.7")
   )
@@
     (property "Reference" "R80" (id 0) (at 63.5 178.7102 90))
     (property "Value" "240R" (id 1) (at 63.5 181.0089 90))
-    (property "Footprint" "" (id 2) (at 63.5 182.88 0)
+    (property "Footprint" "Resistor_SMD:R_0402_1005Metric" (id 2) (at 63.5 182.88 0)
       (effects (font (size 1.27 1.27)) hide)
     )
@@
     (property "Reference" "R82" (id 0) (at 90.17 188.2352 90))
     (property "Value" "10K" (id 1) (at 90.17 184.8189 90))
-    (property "Footprint" "" (id 2) (at 90.17 186.69 0)
+    (property "Footprint" "Resistor_SMD:R_0402_1005Metric" (id 2) (at 90.17 186.69 0)
       (effects (font (size 1.27 1.27)) hide)
     )
@@
     (property "Reference" "R81" (id 0) (at 266.065 178.7102 90))
     (property "Value" "240R" (id 1) (at 266.065 181.0089 90))
-    (property "Footprint" "" (id 2) (at 266.065 182.88 0)
+    (property "Footprint" "Resistor_SMD:R_0402_1005Metric" (id 2) (at 266.065 182.88 0)
       (effects (font (size 1.27 1.27)) hide)
     )
@@
     (property "Reference" "R83" (id 0) (at 285.75 182.5202 90))
     (property "Value" "10K" (id 1) (at 285.75 184.8189 90))
-    (property "Footprint" "" (id 2) (at 285.75 186.69 0)
+    (property "Footprint" "Resistor_SMD:R_0402_1005Metric" (id 2) (at 285.75 186.69 0)
       (effects (font (size 1.27 1.27)) hide)
     )
@@
     (property "Reference" "U9" (id 0) (at 320.04 71.5476 0))
     (property "Value" "VIC-V10" (id 1) (at 320.04 73.8463 0))
-    (property "Footprint" "" (id 2) (at 300.64 70.93 0)
+    (property "Footprint" "BeagleV:JH7100 - BGA-961_31x31_20.5x20.5mm" (id 2) (at 300.64 70.93 0)
       (effects (font (size 1.27 1.27)) hide)
     )
@@
     (property "Reference" "U9" (id 0) (at 124.46 69.0076 0))
     (property "Value" "VIC-V10" (id 1) (at 124.46 71.3063 0))
-    (property "Footprint" "" (id 2) (at 105.06 70.93 0)
-      (effects (font (size 1.27 1.27)) hide)
-    )
+    (property "Footprint" "BeagleV:JH7100 - BGA-961_31x31_20.5x20.5mm" (id 2) (at 105.06 70.93 0)
+      (effects (font (size 1.27 1.27)) hide)
+    )
