File: BeagleV/BeagleV_VIC_HighIF.kicad_sch (KiCad schematic)
At the start: 50 parts, among them U9 VIC-V10, X3 27MHz

Commit message: Initial commit to working branch, Cloned from the gitlab repository
Parts:
- removed P? (x4): VCC_0V9, symbol BeagleV:VCC_0V9
- removed P? (x2): AVDD3V3_USB, symbol BeagleV:AVDD3V3_USB
- C196, C203, C205, C207, C209, C210, C211, C212, C217, C219, C221: footprint (none) -> Capacitor_SMD:C_0201_0603Metric
- C197, C202, C204, C206, C208, C215, C216, C218, C220, C223, C224, C44, C46: footprint (none) -> Capacitor_SMD:C_0402_1005Metric
- D7: footprint (none) -> Diode_SMD:D_SOD-323F
- FB8: footprint (none) -> Inductor_SMD:L_0402_1005Metric_Pad0.77x0.64mm_HandSolder
- R115, R116, R120, R122, R59, R95, R96, R97, R98, R99: footprint (none) -> Resistor_SMD:R_0402_1005Metric
- U9: footprint (none) -> BeagleV:JH7100 - BGA-961_31x31_20.5x20.5mm
- X2: renamed from X?; footprint (none) -> BeagleV:SMCE-3225
- X3: footprint (none) -> BeagleV:SMCE-3225
- gave numbers to parts that had none: 5
Connections:
- net CLK_25M_OUT: now also X2.3; no longer X2.1
- net CLK_27M_OUT: now also X3.3; no longer X3.1
- net GND: now also X2.2, X2.4, X3.2, X3.4; no longer X2.1, X2.3, X3.1, X3.3
- net at C223.1, R122.2: now also X3.1; no longer X3.2
- net at C46.1, R116.2: now also X2.1; no longer X2.2
- net LDO_3V3 renamed VCC_0V9
- net VCC_0V9: no longer C208.1, C209.1, FB8.2, U9.AA23 (AVDD33_USB)
- new net AVDD3V3_USB: C208.1, C209.1, FB8.2, U9.AA23 (AVDD33_USB)
Other:
- moved on the sheet: U9G, U9M
