File: BeagleV/BeagleV_VIC_LCD.kicad_sch (KiCad schematic)
At the start: 46 parts, among them U9 VIC-V10

Commit message: Initial commit to working branch, Cloned from the gitlab repository
Parts:
- C187, C188, C192: footprint (none) -> Capacitor_SMD:C_0402_1005Metric
- C189, C190, C191, C193, C194, C195: footprint (none) -> Capacitor_SMD:C_0201_0603Metric
- R10, R108, R109, R11, R12, R13, R14, R15, R16, R17, R18, R19, R20, R21, R22, R5, R6, R7, R8, R87, R88, R89, R9, R90, R91, R92, R93, R94: footprint (none) -> Resistor_SMD:R_0201_0603Metric
- R240, R241, R242, R243, R244, R245, R246, R247: footprint (none) -> Resistor_SMD:R_0402_1005Metric
- U9: footprint (none) -> BeagleV:JH7100 - BGA-961_31x31_20.5x20.5mm
Other:
- moved on the sheet: U9H, U9K, U9L
