File: BeagleV/BeagleV_Wifi_Bluetooth.kicad_sch (KiCad schematic)
At the start: 42 parts, among them J8 U.FL-R-SMT-1, U12 AP6236, X4 Crystal

Commit message: Initial commit to working branch, Cloned from the gitlab repository
Parts:
- removed P? (x6): 3V3_WIFI, symbol BeagleV:3V3_WIFI
- added C227: 10nF/50V, Capacitor_SMD:C_0402_1005Metric, symbol Device:C_Small
- ANT1: footprint (none) -> BeagleV:RFECA3216060A1T
- C213, C226, C229, C3: footprint (none) -> Capacitor_SMD:C_0201_0603Metric
- C230, C231, C232, C233, C234, C235, C236: footprint (none) -> Capacitor_SMD:C_0402_1005Metric
- FB9: footprint (none) -> Inductor_SMD:L_0402_1005Metric_Pad0.77x0.64mm_HandSolder
- J8: footprint (none) -> BeagleV:U.FL-R-SMT-1
- L2: footprint (none) -> BeagleV:Sunlord_3.0x3.0
- L3: footprint (none) -> Inductor_SMD:L_0201_0603Metric_Pad0.64x0.40mm_HandSolder
- OSC1: footprint (none) -> BeagleV:7XZ-32.768KHz
- R114, R130, R133, R135, R137, R141, R145, R148, R149, R150, R152, R153: footprint (none) -> Resistor_SMD:R_0201_0603Metric
- R136, R139, R140, R154, R155: footprint (none) -> Resistor_SMD:R_0402_1005Metric
- U12: footprint (none) -> BeagleV:AP6236
- X4: footprint (none) -> BeagleV:SMCE-3225
Connections:
- net LDO_3V3 is gone; now on net 3V3_WIFI: C233.1, C234.1, C3.1, FB9.2, OSC1.1 (EN), OSC1.4 (VDD), R130.1, R137.2, R141.1, U12.22 (VDDIO)
- net GND: now also C227.1; no longer ANT1.3
- net 3V3_WIFI: now reaches C229.1, C230.1, C231.1, U12.9 (VBAT)
- new net: ANT1.3, C227.2
