File: BeagleV/VIC_Power.kicad_sch (KiCad schematic)
At the start: 74 parts, among them U9 VIC-V10

Commit message: Initial commit to working branch, Cloned from the gitlab repository
Parts:
- removed P? (x5): VCC_0V9, symbol BeagleV:VCC_0V9
- removed P? (x2): AVDD09_PLL, symbol BeagleV:AVDD09_PLL
- C112, C113, C114, C115, C117, C118, C119, C124, C125, C126, C127, C128, C129, C130, C131, C132, C137, C138, C139, C140, C146, C147, C148, C149, C150, C151, C152, C153, C154, C161, C162, C163, C164, C165, C166, C167, C168, C169, C170, C171, C172, C173, C174, C175: footprint (none) -> Capacitor_SMD:C_0201_0603Metric
- C116, C121, C122, C123, C133, C135, C136, C141, C143, C144, C145, C155, C158, C159, C160, C176: footprint (none) -> Capacitor_SMD:C_0402_1005Metric
- C120, C134, C142, C156, C157: footprint (none) -> Capacitor_SMD:C_0603_1608Metric
- FB7: footprint (none) -> Inductor_SMD:L_0402_1005Metric_Pad0.77x0.64mm_HandSolder
- U9: footprint (none) -> BeagleV:JH7100 - BGA-961_31x31_20.5x20.5mm
Connections:
- net AVDD09_PLL: now reaches C116.1, C117.1, C118.1, C119.1, FB7.1
- net AVDD09_PLL: now also U9.U21 (AVDD09_PLL0), U9.U22 (AVDD09_PLL1), U9.V21 (AVDD09_PLL2)
- net LDO_3V3 renamed VCC_0V9
Other:
- moved on the sheet: U9A, U9C, U9D
